File: Inda_Kidcad/Inda_Kidcad.kicad_pcb (KiCad board)
At the start: 2 copper layers, 88.5 x 71 mm, 152 parts, among them J1 SERIALWIRE, J10 Conn_01x03_Pin, J11 Conn_01x04_Pin, J12 Conn_01x04_Pin, J13 Conn_01x04_Pin, J14 Conn_01x04_Pin, J15 Conn_01x02_Pin, J16 Conn_01x01_Pin, J17 Conn_01x01_Pin, J19 Conn_01x02_Pin, J2 LIPO, J20 Conn_01x02_Pin, J21 Conn_01x03_Pin, J22 Conn_01x03_Pin, J23 Conn_01x02_Pin, J24 Conn_01x02_Pin, J25 Conn_01x02_Pin, J3 BRIDGE, J4 Conn_01x03_Pin, J5 Conn_01x03_Pin, J6 Conn_01x03_Pin, J7 Conn_01x03_Pin, J8 Conn_01x02_Pin, J9 Conn_01x02_Pin, Q1 AO3400A, Q2 AO3400A, Q3 AO3400A, Q4 AO3400A, Q5 AO3401A, Q6 AO3401A, SW1 SW_Push, SW2 SW_Push, SW3 SW_Push_SPDT, SW4 SW_Push, SW5 SW_Push, SW6 SW_Push, U1 STM32f103C8t6, U10 QRE111GR, U11 QRE111GR, U12 vs1838, U2 DRV8833, U3 AD8418, U4 AD8418, U5 DRV8833, U6 CN3903, U7 AMS1117-5.0, U8 QRE111GR, U9 QRE111GR, Y2 8Mhz

Commit message: codigo funciona 1
Parts:
- R43: value 47K -> 36k
