File: Inda_Kidcad/Inda_Kidcad.kicad_pcb (KiCad board)
At the start: 2 copper layers, 88.5 x 71 mm, 152 parts, among them J1 SERIALWIRE, J10 Conn_01x03_Pin, J11 Conn_01x04_Pin, J12 Conn_01x04_Pin, J13 Conn_01x04_Pin, J14 Conn_01x04_Pin, J15 Conn_01x02_Pin, J16 Conn_01x01_Pin, J17 Conn_01x01_Pin, J19 Conn_01x02_Pin, J2 LIPO, J20 Conn_01x02_Pin, J21 Conn_01x03_Pin, J22 Conn_01x03_Pin, J23 Conn_01x02_Pin, J24 Conn_01x02_Pin, J25 Conn_01x02_Pin, J3 BRIDGE, J4 Conn_01x03_Pin, J5 Conn_01x03_Pin, J6 Conn_01x03_Pin, J7 Conn_01x03_Pin, J8 Conn_01x02_Pin, J9 Conn_01x02_Pin, Q1 AO3400A, Q2 AO3400A, Q3 AO3400A, Q4 AO3400A, Q5 AO3401A, Q6 AO3401A, SW1 SW_Push, SW2 SW_Push, SW3 SW_Push_SPDT, SW4 SW_Push, SW5 SW_Push, SW6 SW_Push, U1 STM32f103C8t6, U10 QRE111GR, U11 QRE111GR, U12 vs1838, U2 DRV8833, U3 AD8418, U4 AD8418, U5 DRV8833, U6 CN3903, U7 AMS1117-5.0, U8 QRE111GR, U9 QRE111GR, Y2 8Mhz

Commit message: Version 2 De Sumo Inda
Parts:
- removed C16, C18, C20, C22: 10uF, Capacitor_SMD:C_0603_1608Metric_Pad1.08x0.95mm_HandSolder
- removed C17, C19, C21, C23: 100nF, Capacitor_SMD:C_0603_1608Metric_Pad1.08x0.95mm_HandSolder
- removed C24, C25, C27: 100nF, Capacitor_SMD:C_0603_1608Metric
- removed C26: 22uF, Capacitor_SMD:C_0603_1608Metric
- removed C28: 10uF, Capacitor_SMD:CP_Elec_4x5.8
- removed C29, C30: 10uF, Capacitor_SMD:C_1206_3216Metric_Pad1.33x1.80mm_HandSolder
- removed D1, D2, D3, D4: SFH4546, Footprint:SFH4545_LED
- removed G*** (x2): LOGO, LOGO
- removed J11, J12, J13, J14: Conn_01x04_Pin, Footprint:CONN_SMD_01X04_IR
- removed J16, J17: Conn_01x01_Pin, Footprint:pad_1_SMD
- removed J2: LIPO, Connector_Molex:Molex_SL_171971-0002_1x02_P2.54mm_Vertical
- removed J24: Conn_01x02_Pin, Footprint:CONN_SMD_01X02_IR
- removed JP1: Jumper_3_Open, Jumper:SolderJumper-3_P1.3mm_Open_Pad1.0x1.5mm_NumberLabels
- removed L1, L2, L3, L4: TEFT4300, Footprint:TEFT4300_LED
- removed L5: 4.7uH, Inductor_SMD:L_Wuerth_HCM-7050
- removed Q1, Q2, Q3, Q4: AO3400A, Package_TO_SOT_SMD:SOT-23
- removed R10, R13, R16, R8: 33, Resistor_SMD:R_0805_2012Metric_Pad1.20x1.40mm_HandSolder
- removed R11, R14, R17, R7: 3.3K, Resistor_SMD:R_0805_2012Metric_Pad1.20x1.40mm_HandSolder
- removed R12, R15, R6, R9: 10K, Resistor_SMD:R_0805_2012Metric_Pad1.20x1.40mm_HandSolder
- removed R30: 150, Resistor_SMD:R_0805_2012Metric_Pad1.20x1.40mm_HandSolder
- removed R31: 15k, Resistor_SMD:R_0805_2012Metric_Pad1.20x1.40mm_HandSolder
- removed R4, R5: 0.05, Resistor_SMD:R_2512_6332Metric_Pad1.40x3.35mm_HandSolder
- removed U11: QRE111GR, Footprint:QRE1113GR_IR
- removed U6: CN3903, Package_SO:HSOP-8-1EP_3.9x4.9mm_P1.27mm_EP2.41x3.1mm
- removed U7: AMS1117-5.0, Package_TO_SOT_SMD:SOT-223-3_TabPin2
- added C39: 0.1uF, Capacitor_SMD:C_0603_1608Metric, F.Cu at (137.5, 156.1)
- added C40: 22uF, Capacitor_SMD:C_0603_1608Metric, F.Cu at (137.5, 158.6)
- added C41: 22uF, Capacitor_SMD:C_0603_1608Metric, F.Cu at (137.5, 161.1)
- added C42: 22uF, Capacitor_SMD:C_0603_1608Metric, F.Cu at (137.5, 163.6)
- added C43: 22uF, Capacitor_SMD:C_0603_1608Metric, F.Cu at (137.5, 166.1)
- C11, C12, C13, C14, C31, C32, C8, C9, J10, J15, J19, J20, J23, J25, J4, J5, J6, J8, J9, R1, R2, R3, R42, R43: moved to F.Cu
- C36: value 100nF -> 22uF; footprint Capacitor_SMD:C_0603_1608Metric_Pad1.08x0.95mm_HandSolder -> Capacitor_SMD:C_0603_1608Metric
- J7: value Conn_01x03_Pin -> XT30; footprint Footprint:CONN_SMD_01X03_IR -> Connector_AMASS:AMASS_XT30U-F_1x02_P5.0mm_Vertical; moved to F.Cu
- R21: value 18k -> 200K; footprint Resistor_SMD:R_0805_2012Metric_Pad1.20x1.40mm_HandSolder -> Resistor_SMD:R_0603_1608Metric_Pad0.98x0.95mm_HandSolder
- R22: value 100K -> 116K; footprint Resistor_SMD:R_0805_2012Metric_Pad1.20x1.40mm_HandSolder -> Resistor_SMD:R_0603_1608Metric_Pad0.98x0.95mm_HandSolder
- R23: value 39k -> 22K; footprint Resistor_SMD:R_0805_2012Metric_Pad1.20x1.40mm_HandSolder -> Resistor_SMD:R_0603_1608Metric_Pad0.98x0.95mm_HandSolder
- U3: value AD8418 -> AP2112K-3.3TRG1; footprint Footprint:AD8418_soic -> Package_TO_SOT_SMD:SOT-23-5
- U4: value AD8418 -> MSTPS563200DDCR; footprint Footprint:AD8418_soic -> Package_TO_SOT_SMD:SOT-23-6
- moved C12 186.3 mm to (255.6, 134.2), turned to 0 degrees
- moved C11 184.2 mm to (255.6, 131.7), turned to 0 degrees
- moved C10 182.3 mm to (247.5, 145.9), turned to 0 degrees
- moved J5 182.2 mm to (267.7, 95.7)
- moved C33 180.5 mm to (265.9, 103.6), turned to 0 degrees
- moved U2 178.2 mm to (248.9, 133.7), turned to 0 degrees
- moved U8 175.0 mm to (260.3, 91.0), turned to 0 degrees
- moved R41 173.3 mm to (242.6, 110.3), turned to 0 degrees
- moved C13 172.9 mm to (255.6, 136.7), turned to 0 degrees
- moved C37 172.9 mm to (246.7, 123.3), turned to 0 degrees
- moved R25 172.1 mm to (254.4, 92.9), turned to 0 degrees
- moved U12 172.0 mm to (242.2, 119.9), turned to 0 degrees
- moved R40 171.5 mm to (242.6, 107.3), turned to 0 degrees
- moved C14 171.1 mm to (255.6, 139.2), turned to 0 degrees
- moved C38 170.9 mm to (246.7, 125.9), turned to 0 degrees
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Connections:
- net /MOTA_L renamed /MOTOR/MOTA_L
- net /MOTA_R renamed /MOTOR/MOTA_R
- net /Mod_TX4 renamed Net-(U1-PB2)
- net /sensores_linea/CONN1_3V3 renamed /SENSOR_LINEA/CONN1_3V3
- net /sensores_linea/CONN1_GND renamed /SENSOR_LINEA/CONN1_GND
- net /sensores_linea/CONN2_3V3 renamed /SENSOR_LINEA/CONN2_3V3
- net /sensores_linea/CONN2_GND renamed /SENSOR_LINEA/CONN2_GND
- net /sensores_linea/CONN3_3V3 renamed /SENSOR_LINEA/CONN3_3V3
- net /sensores_linea/CONN3_GND renamed /SENSOR_LINEA/CONN3_GND
- net /sensores_linea/CONN_IR1 renamed /SENSOR_LINEA/CONN_IR1
- net /sensores_linea/CONN_IR2 renamed /SENSOR_LINEA/CONN_IR2
- net /sensores_linea/CONN_IR3 renamed /SENSOR_LINEA/CONN_IR3
- C31 pad 1: /VBAT -> /ALIMENTACION/VBAT
- C32 pad 2: /VBAT -> /ALIMENTACION/VBAT
- C36 pad 1: /sensores_linea/CONN4_3V3 -> GND
- C36 pad 2: /sensores_linea/CONN4_GND -> Net-(U4-VIN)
- J19 pad 1: /MOTB_L -> /MOTOR/MOTB_L
- J20 pad 1: /MOTB_R -> /MOTOR/MOTB_R
- J3 pad 1: /VBAT -> /ALIMENTACION/VBAT
- J3 pad 2: /++ -> Net-(J3-Pin_2)
- J7 pad 1: /sensores_linea/CONN_IR4 -> GND
- J7 pad 2: /sensores_linea/CONN4_3V3 -> Net-(J3-Pin_2)
- Q5 pad 3: /++ -> Net-(J3-Pin_2)
- Q6 pad 3: /VBAT -> /ALIMENTACION/VBAT
- R20 pad 1: /VBAT -> /ALIMENTACION/VBAT
- R21 pad 1: /VBAT -> Net-(U4-EN)
- R21 pad 2: Net-(U6-EN) -> /ALIMENTACION/VBAT
- R22 pad 1: /ALIMENTACION/FB -> +5V
- R22 pad 2: +3.3V -> Net-(U4-FB)
- R23 pad 1: GND -> Net-(U4-FB)
- R23 pad 2: /ALIMENTACION/FB -> GND
- U1 pad 13: /Mod_RX4 -> unconnected-(U1-PA3_ADC3_RX2_PWM2-Pad13)
- U1 pad 15: /CURRENT_MOTL -> unconnected-(U1-PA5_ADC5_SCK1-Pad15)
- U1 pad 16: /CURRENT_MOTR -> unconnected-(U1-PA6_ADC6_MISO1_PWM3-Pad16)
- U2 pad 4: /Motores/SEN_MOTR -> /MOTOR/MOTB_R
- U2 pad 5: /Motores/SEN_MOTR -> /MOTOR/MOTB_R
- U3 pad 1: /MOTB_R -> +5V
- U3 pad 3: GND -> +5V
- U3 pad 5: /CURRENT_MOTR -> +3.3V
- U4 pad 1: /MOTB_L -> GND
- U4 pad 2: GND -> Net-(U4-SW)
- U4 pad 3: GND -> Net-(U4-VIN)
- U4 pad 4: unconnected-(U4-NC-Pad4) -> Net-(U4-FB)
- U4 pad 5: /CURRENT_MOTL -> Net-(U4-EN)
- U4 pad 6: /Motores/vcc -> Net-(U4-BST)
- U5 pad 4: /Motores/SEN_MOTL -> /MOTOR/MOTB_L
- U5 pad 5: /Motores/SEN_MOTL -> /MOTOR/MOTB_L
Routing:
- net GND: track 697.6 -> 0.00 mm, vias 115 -> 0
- net +3.3V: track 224.5 -> 0.00 mm, vias 23 -> 0
- net /VBAT: track 214.2 -> 0.00 mm, vias 52 -> 0
- net /EN_MOT: track 81.1 -> 0.00 mm, vias 3 -> 0
- net /PWMA_MOTR: track 65.1 -> 0.00 mm
- net /PWMB_MOTR: track 64.3 -> 0.00 mm, vias 2 -> 0
- net /PWMB_MOTL: track 60.6 -> 0.00 mm, vias 2 -> 0
- net /CURRENT_MOTR: track 58.6 -> 0.00 mm, vias 6 -> 0
- net /PWMA_MOTL: track 55.2 -> 0.00 mm
- net Net-(U1-PB2): track 55.0 -> 0.00 mm, vias 2 -> 0
- net /BOOT0: track 47.5 -> 0.00 mm, vias 4 -> 0
- net +5V: track 47.2 -> 0.00 mm, vias 2 -> 0
- net /Motores/vcc: track 45.2 -> 0.00 mm, vias 3 -> 0
- net /IR_38khz: track 44.2 -> 0.00 mm, vias 2 -> 0
- net /CURRENT_MOTL: track 38.8 -> 0.00 mm, vias 2 -> 0
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- removed copper zone on B.Cu, net GND
- removed copper zone on F.Cu, net GND
Other:
- board size 88.5 x 71 mm -> 88 x 55.2 mm
- board text removed: "+"
- board text removed: "-"
- board text removed: "3v"
- board text removed: "5v"
- board text removed: "KARANE"
- board text removed: "L1"
- board text removed: "L2"
- board text removed: "L3"
- board text removed: "M1"
- board text removed: "M2"
- board text removed: "Rx"
- board text removed: "Tx"
- board text removed: "boot"
- board text removed: "clk"
- board text removed: "dio"
- board text removed: "ir"
- board text removed: "nrst"
- board text removed: "rx1"
- board text removed: "rx2"
- board text removed: "rx3"
- board text removed: "rx4"
- board text removed: "tx1"
- board text removed: "tx2"
- board text removed: "tx3"
- board text removed: "tx4"

Commit message: Se cambia simbolos como huellas, se coloca solo mosfet para interruptor y se empieza con pcb
Parts:
- removed C31: 10uF, Capacitor_Tantalum_SMD:CP_EIA-3528-15_AVX-H_HandSolder
- removed C32, C33, C34, C35: 100nF, Capacitor_SMD:C_0603_1608Metric
- removed C36, C40, C41, C42, C43: 22uF, Capacitor_SMD:C_0603_1608Metric
- removed C37: 100nF, Capacitor_SMD:C_0603_1608Metric_Pad1.08x0.95mm_HandSolder
- removed C38: 10uF, Capacitor_SMD:C_0603_1608Metric_Pad1.08x0.95mm_HandSolder
- removed C39: 0.1uF, Capacitor_SMD:C_0603_1608Metric
- removed D10, D7, D8, D9: LED, LED_SMD:LED_1206_3216Metric_Pad1.42x1.75mm_HandSolder
- removed J19, J20: Conn_01x02_Pin, Footprint:Molex Header 2 hole 2.54mm
- removed J21, J22: Conn_01x03_Pin, Connector_PinHeader_2.54mm:PinHeader_1x03_P2.54mm_Vertical
- removed J23, J25, J8, J9: Conn_01x02_Pin, Footprint:CONN_SMD_01X02_IR
- removed J4, J6: Conn_01x03_Pin, Footprint:CONN_SMD_01X03_IR
- removed J7: XT30, Connector_AMASS:AMASS_XT30U-F_1x02_P5.0mm_Vertical
- removed Q5, Q6: AO3401A, Package_TO_SOT_SMD:SOT-23
- removed R29: 15k, Resistor_SMD:R_0805_2012Metric_Pad1.20x1.40mm_HandSolder
- removed R32, R33, R34, R35: 2.2K, Resistor_SMD:R_0805_2012Metric_Pad1.20x1.40mm_HandSolder
- removed R36, R42: 100K, Resistor_SMD:R_0805_2012Metric_Pad1.20x1.40mm_HandSolder
- removed R37: 20K, Resistor_SMD:R_0805_2012Metric_Pad1.20x1.40mm_HandSolder
- removed R38: 1K, Resistor_SMD:R_0805_2012Metric_Pad1.20x1.40mm_HandSolder
- removed R39: 47K, Resistor_SMD:R_0805_2012Metric_Pad1.20x1.40mm_HandSolder
- removed R40: 100, Resistor_SMD:R_0805_2012Metric_Pad1.20x1.40mm_HandSolder
- removed R41: 10k, Resistor_SMD:R_0805_2012Metric_Pad1.20x1.40mm_HandSolder
- removed R43: 36k, Resistor_SMD:R_0805_2012Metric_Pad1.20x1.40mm_HandSolder
- removed U12: vs1838, Connector_PinHeader_2.54mm:PinHeader_1x03_P2.54mm_Vertical
- removed Y2: 8Mhz, Crystal:Crystal_SMD_Abracon_ABM8AIG-4Pin_3.2x2.5mm
- added C16: 100nF, Capacitor_SMD:C_0805_2012Metric_Pad1.18x1.45mm_HandSolder, F.Cu at (111.0, 138.8)
- added C17: 10uF, Capacitor_Tantalum_SMD:CP_EIA-3528-21_Kemet-B_HandSolder, F.Cu at (110.2, 135.8)
- added C18: 10uF, Capacitor_Tantalum_SMD:CP_EIA-3528-15_AVX-H_HandSolder, F.Cu at (158.1, 125.6)
- added C19: 100nF, Capacitor_SMD:C_0603_1608Metric, F.Cu at (156.9, 122.6)
- added C20: 22uF, Capacitor_SMD:C_0603_1608Metric, F.Cu at (249.5, 143.9)
- added C21: 22uF, Capacitor_SMD:C_0603_1608Metric, F.Cu at (249.5, 146.4)
- added C22: 0.1uF, Capacitor_SMD:C_0603_1608Metric, F.Cu at (166.3, 113.5)
- added C23: 22uF, Capacitor_SMD:C_0603_1608Metric, F.Cu at (153.0, 116.5)
- added C26: 100nF, Capacitor_SMD:C_0603_1608Metric, F.Cu at (301.5, 110.6)
- added C27: 100nF, Capacitor_SMD:C_0603_1608Metric, F.Cu at (301.5, 113.1)
- added C28: 100nF, Capacitor_SMD:C_0603_1608Metric, F.Cu at (301.5, 115.6)
- added C29: 22uF, Capacitor_Tantalum_SMD:CP_EIA-3528-15_AVX-H_HandSolder, F.Cu at (165.1, 120.6)
- added C30: 22uF, Capacitor_Tantalum_SMD:CP_EIA-3528-15_AVX-H_HandSolder, F.Cu at (156.0, 115.5)
- added D1: LED, LED_SMD:LED_1206_3216Metric_Pad1.42x1.75mm_HandSolder, F.Cu at (279.6, 114.5)
- added D2: LED, LED_SMD:LED_1206_3216Metric_Pad1.42x1.75mm_HandSolder, F.Cu at (279.6, 117.9)
- added D3: LED, LED_SMD:LED_1206_3216Metric_Pad1.42x1.75mm_HandSolder, F.Cu at (279.6, 121.3)
- added D4: LED, LED_SMD:LED_1206_3216Metric_Pad1.42x1.75mm_HandSolder, F.Cu at (279.6, 124.7)
- added J11: CONN_ML, Footprint:Molex Header 2 hole 2.54mm, F.Cu at (119.0, 135.5)
- added J12: XT30, Footprint:XT30_H_M, B.Cu at (167.5, 130.5)
- added J13: Conn_01x03_Pin, Footprint:CONN_SMD_01X03_IR, F.Cu at (303.3, 98.0)
- added J14: Conn_01x03_Pin, Footprint:CONN_SMD_01X03_IR, F.Cu at (303.3, 102.7)
- added JP1: JUMPER_MODE_MR, Jumper:SolderJumper-3_P1.3mm_Open_RoundedPad1.0x1.5mm, B.Cu at (147.0, 139.0)
- added JP2: JUMPER_MODE_ML, Jumper:SolderJumper-3_P1.3mm_Open_RoundedPad1.0x1.5mm, B.Cu at (108.5, 131.8)
- added L1: 3.3uH, Inductor_SMD:L_Sunlord_MWSA0402S, F.Cu at (160.5, 115.5)
- added R10: 2.2K, Resistor_SMD:R_0805_2012Metric_Pad1.20x1.40mm_HandSolder, F.Cu at (269.5, 123.2)
- added R11: 20K, Resistor_SMD:R_0805_2012Metric_Pad1.20x1.40mm_HandSolder, F.Cu at (274.2, 114.3)
- added R12: 1K, Resistor_SMD:R_0805_2012Metric_Pad1.20x1.40mm_HandSolder, F.Cu at (274.2, 117.3)
- added R13: 47k, Capacitor_SMD:C_0805_2012Metric_Pad1.18x1.45mm_HandSolder, F.Cu at (254.5, 128.8)
- added R14: 100, Resistor_SMD:R_0805_2012Metric_Pad1.20x1.40mm_HandSolder, F.Cu at (274.2, 120.2)
- added R15: 10k, Resistor_SMD:R_0805_2012Metric_Pad1.20x1.40mm_HandSolder, F.Cu at (274.2, 123.2)
- added R17: 100K, Resistor_SMD:R_0805_2012Metric_Pad1.20x1.40mm_HandSolder, F.Cu at (158.8, 134.7)
- added R4: 36k, Resistor_SMD:R_0805_2012Metric_Pad1.20x1.40mm_HandSolder, F.Cu at (264.7, 117.3)
- added R5: 2.2K, Resistor_SMD:R_0805_2012Metric_Pad1.20x1.40mm_HandSolder, F.Cu at (264.7, 120.2)
- added R6: 2.2K, Resistor_SMD:R_0805_2012Metric_Pad1.20x1.40mm_HandSolder, F.Cu at (264.7, 123.2)
- added R7: 100K, Resistor_SMD:R_0805_2012Metric_Pad1.20x1.40mm_HandSolder, F.Cu at (269.5, 114.3)
- added R8: 47K, Resistor_SMD:R_0805_2012Metric_Pad1.20x1.40mm_HandSolder, F.Cu at (269.5, 117.3)
- added R9: 2.2K, Resistor_SMD:R_0805_2012Metric_Pad1.20x1.40mm_HandSolder, F.Cu at (269.5, 120.2)
- added U6: AP2112K-3.3TRG1, Package_TO_SOT_SMD:SOT-23-5, F.Cu at (254.1, 149.5)
- added U7: MSTPS563200DDCR, Package_TO_SOT_SMD:SOT-23-6, F.Cu at (165.5, 116.5)
- added Y1: 8Mhz, Crystal:Crystal_SMD_Abracon_ABM8AIG-4Pin_3.2x2.5mm, F.Cu at (273.1, 126.9)
- C1, C4: value 100nF -> 1nF
- C10: value 10uF -> 100nF; footprint Capacitor_Tantalum_SMD:CP_EIA-3528-21_Kemet-B_HandSolder -> Capacitor_SMD:C_0603_1608Metric_Pad1.08x0.95mm_HandSolder
- C11: value 10nF -> 10uF
- C12, C13: value 2.2uF -> 100nF; footprint Capacitor_SMD:C_0603_1608Metric_Pad1.08x0.95mm_HandSolder -> Capacitor_SMD:C_0805_2012Metric_Pad1.18x1.45mm_HandSolder
- C14: value 10nF -> 10uF; footprint Capacitor_SMD:C_0603_1608Metric_Pad1.08x0.95mm_HandSolder -> Capacitor_Tantalum_SMD:CP_EIA-3528-21_Kemet-B_HandSolder
- C15: value 10uF -> 100nF; footprint Capacitor_Tantalum_SMD:CP_EIA-3528-21_Kemet-B_HandSolder -> Capacitor_SMD:C_0805_2012Metric_Pad1.18x1.45mm_HandSolder
- C2, C3: value 100nF -> 20pF
- C5, C7: value 20pF -> 100nF
- C8, C9: value 1nF -> 100nF
- J1: value SERIALWIRE -> SWD_UART_CONN
- J10: value Conn_01x03_Pin -> CONN_MR; footprint Footprint:CONN_SMD_01X03_IR -> Footprint:Molex Header 2 hole 2.54mm
- J15: value Conn_01x02_Pin -> Conn_01x03_Pin; footprint Footprint:CONN_SMD_01X02_IR -> Footprint:CONN_SMD_01X03_IR
- J3: value BRIDGE -> Conn_01x03; footprint Connector_PinHeader_2.54mm:PinHeader_1x02_P2.54mm_Vertical -> Connector_PinHeader_2.54mm:PinHeader_1x03_P2.54mm_Vertical
- J5: value Conn_01x03_Pin -> SQJ951EP; footprint Footprint:CONN_SMD_01X03_IR -> Package_SO:PowerPAK_SO-8_Dual
- R18: value 100K -> 10k
- R19: value 100K -> 200K; footprint Resistor_SMD:R_0805_2012Metric_Pad1.20x1.40mm_HandSolder -> Resistor_SMD:R_0603_1608Metric_Pad0.98x0.95mm_HandSolder
- R20: value 20K -> 100k; footprint Resistor_SMD:R_0805_2012Metric_Pad1.20x1.40mm_HandSolder -> Resistor_SMD:R_0603_1608Metric_Pad0.98x0.95mm_HandSolder
- R21: value 200K -> 22K
- R22: value 116K -> 150; footprint Resistor_SMD:R_0603_1608Metric_Pad0.98x0.95mm_HandSolder -> Resistor_SMD:R_0805_2012Metric_Pad1.20x1.40mm_HandSolder
- R23: value 22K -> 15k; footprint Resistor_SMD:R_0603_1608Metric_Pad0.98x0.95mm_HandSolder -> Resistor_SMD:R_0805_2012Metric_Pad1.20x1.40mm_HandSolder
- R28: value 150 -> 15k; footprint Resistor_SMD:R_0805_2012Metric_Pad1.20x1.40mm_HandSolder -> Resistor_SMD:R_0603_1608Metric_Pad0.98x0.95mm_HandSolder
- R3: value 47k -> 100K; footprint Capacitor_SMD:C_0805_2012Metric_Pad1.18x1.45mm_HandSolder -> Resistor_SMD:R_0805_2012Metric_Pad1.20x1.40mm_HandSolder
- SW3: value SW_Push_SPDT -> SW_Push; footprint Button_Switch_SMD:SW_SPDT_PCM12 -> Button_Switch_SMD:SW_SPST_CK_RS282G05A3
- SW6: value SW_Push -> SW_Push_SPDT; footprint Button_Switch_SMD:SW_SPST_CK_RS282G05A3 -> Button_Switch_SMD:SW_SPDT_PCM12
- U2: value DRV8833 -> vs1838; footprint Footprint:drv8833 -> Footprint:1838_aliexpress
- U3: value AP2112K-3.3TRG1 -> DRV8212DSGR; footprint Package_TO_SOT_SMD:SOT-23-5 -> Package_SON:WSON-8-1EP_2x2mm_P0.5mm_EP0.9x1.6mm
- U4: value MSTPS563200DDCR -> DRV8212DSGR; footprint Package_TO_SOT_SMD:SOT-23-6 -> Package_SON:WSON-8-1EP_2x2mm_P0.5mm_EP0.9x1.6mm
- U5: value DRV8833 -> ~; footprint Footprint:drv8833 -> Footprint:BRIDGE_2P; moved to B.Cu
- moved R22 160.7 mm to (290.1, 97.0)
- moved R23 160.6 mm to (290.1, 99.9)
- moved C15 140.2 mm to (108.5, 131.8), turned to -90 degrees
- moved SW3 117.3 mm to (252.9, 108.4)
- moved J5 115.9 mm to (157.1, 130.4), turned to 180 degrees
- moved C13 112.7 mm to (143.0, 132.0), turned to 180 degrees
- moved J10 112.3 mm to (135.0, 135.0), turned to 90 degrees
- moved C14 111.7 mm to (144.0, 135.0)
- moved C12 108.8 mm to (147.0, 139.0), turned to 90 degrees
- moved J3 108.3 mm to (249.8, 123.5)
- moved R28 92.9 mm to (162.0, 110.5), turned to -90 degrees
- moved U5 84.5 mm to (166.0, 124.0), turned to 180 degrees
- moved J15 81.8 mm to (303.3, 107.2)
- moved R20 64.8 mm to (160.0, 110.5), turned to 90 degrees
- moved SW6 60.3 mm to (160.5, 139.0)
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Connections:
- C1 pad 1: +3.3V -> /NRST
- C10 pad 1: /VBAT -> Net-(U2-vcc)
- C11 pad 1: Net-(U2-VCP) -> Net-(U2-vcc)
- C11 pad 2: /VBAT -> GND
- C12 pad 1: Net-(U2-VINT) -> GND
- C12 pad 2: GND -> +3.3V
- C13 pad 1: Net-(U5-VINT) -> GND
- C13 pad 2: GND -> /VBAT
- C14 pad 1: Net-(U5-VCP) -> /VBAT
- C14 pad 2: /VBAT -> GND
- C15 pad 1: /VBAT -> GND
- C15 pad 2: GND -> +3.3V
- C2 pad 1: +3.3V -> /OSC_B
- C3 pad 1: +3.3V -> /OSC_A
- C4 pad 1: +3.3V -> /BOOT0
- C5 pad 1: /OSC_B -> +3.3V
- C7 pad 1: /OSC_A -> +3.3V
- C8 pad 1: /NRST -> +3.3V
- C9 pad 1: /BOOT0 -> +3.3V
- J10 pad 1: /Linea3 -> /MOTOR/MOTA_R
- J10 pad 2: /Linea2 -> /MOTOR/MOTB_R
- J15 pad 1: +3.3V -> /SENSOR_LINEA/CONN_IR3
- J15 pad 2: GND -> /SENSOR_LINEA/CONN3_3V3
- J3 pad 1: /ALIMENTACION/VBAT -> GND
- J3 pad 2: Net-(J3-Pin_2) -> +5V
- J5 pad 1: /SENSOR_LINEA/CONN_IR1 -> Net-(D5-K)
- J5 pad 2: /SENSOR_LINEA/CONN1_3V3 -> Net-(D5-A)
- J5 pad 3: /SENSOR_LINEA/CONN1_GND -> Net-(D5-K)
- R18 pad 1: Net-(D5-K) -> /VBAT
- R18 pad 2: Net-(SW3-A) -> Net-(D6-A)
- R19 pad 1: Net-(D5-A) -> Net-(U7-EN)
- R19 pad 2: Net-(SW3-A) -> /VBAT
- R20 pad 1: /ALIMENTACION/VBAT -> +5V
- R20 pad 2: Net-(D6-A) -> Net-(R20-Pad2)
- R21 pad 1: Net-(U4-EN) -> Net-(U7-FB)
- R21 pad 2: /ALIMENTACION/VBAT -> GND
- R22 pad 1: +5V -> /SENSOR_LINEA/CONN1_3V3
- R22 pad 2: Net-(U4-FB) -> Net-(U8-A)
- R23 pad 1: Net-(U4-FB) -> /SENSOR_LINEA/CONN1_3V3
- R23 pad 2: GND -> /SENSOR_LINEA/CONN_IR1
- R24 pad 1: /SENSOR_LINEA/CONN1_3V3 -> /SENSOR_LINEA/CONN2_3V3
- R24 pad 2: Net-(U8-A) -> Net-(U9-A)
- R25 pad 1: /SENSOR_LINEA/CONN1_3V3 -> /SENSOR_LINEA/CONN2_3V3
- R25 pad 2: /SENSOR_LINEA/CONN_IR1 -> /SENSOR_LINEA/CONN_IR2
- R26 pad 1: /SENSOR_LINEA/CONN2_3V3 -> /SENSOR_LINEA/CONN3_3V3
- R26 pad 2: Net-(U9-A) -> Net-(U10-A)
- R27 pad 1: /SENSOR_LINEA/CONN2_3V3 -> /SENSOR_LINEA/CONN3_3V3
- R27 pad 2: /SENSOR_LINEA/CONN_IR2 -> /SENSOR_LINEA/CONN_IR3
- R28 pad 1: /SENSOR_LINEA/CONN3_3V3 -> Net-(R20-Pad2)
- R28 pad 2: Net-(U10-A) -> Net-(U7-FB)
- R3 pad 1: Net-(U1-PB2) -> /VBAT
- R3 pad 2: GND -> /VOLTAGE
- SW3 pad 1: Net-(SW3-A) -> Net-(R7-Pad1)
- SW3 pad 2: GND -> +3.3V
- SW6 pad 2: +3.3V -> GND
- U1 pad 10: /Mod_RX1 -> /SHARP_A1
- U1 pad 11: /Mod_RX2 -> /SHARP_A2
- U1 pad 12: /Mod_RX3 -> /SHARP_A3
- U1 pad 13: unconnected-(U1-PA3_ADC3_RX2_PWM2-Pad13) -> /SHARP_A4
- U1 pad 25: /Mod_TX1 -> unconnected-(U1-PB12_SS2-Pad25)
- U1 pad 33: /EN_MOT -> unconnected-(U1-PA12_USB++-Pad33)
- U2 pad 1: /EN_MOT -> /IR_38khz
- U2 pad 2: /MOTOR/MOTA_R -> GND
- U2 pad 3: GND -> Net-(U2-vcc)
- U3 pad 1: +5V -> /VBAT
- U3 pad 2: GND -> /MOTOR/MOTA_R
- U3 pad 3: +5V -> /MOTOR/MOTB_R
- U3 pad 4: unconnected-(U3-NC-Pad4) -> GND
- U3 pad 5: +3.3V -> /PWMB_MOTR
- U4 pad 1: GND -> /VBAT
- U4 pad 2: Net-(U4-SW) -> /MOTOR/MOTB_L
- U4 pad 3: Net-(U4-VIN) -> /MOTOR/MOTA_L
- U4 pad 4: Net-(U4-FB) -> GND
- U4 pad 5: Net-(U4-EN) -> /PWMB_MOTL
- U4 pad 6: Net-(U4-BST) -> /PWMA_MOTL
- U5 pad 1: /EN_MOT -> Net-(D5-K)
- U5 pad 2: /MOTOR/MOTA_L -> /VBAT
Routing:
- net Net-(U7-FB): track 0.00 -> 9.61 mm, vias 0 -> 2
- net Net-(D5-A): track 0.00 -> 9.52 mm, vias 0 -> 3
- net /VBAT: track 0.00 -> 4.25 mm, vias 0 -> 29
- net Net-(D5-K): track 0.00 -> 4.01 mm
- net Net-(U7-SW): track 0.00 -> 3.87 mm
- net Net-(SW6-A): track 0.00 -> 3.06 mm
- net Net-(U7-EN): track 0.00 -> 2.74 mm
- net +5V: track 0.00 -> 2.44 mm, vias 0 -> 10
- net Net-(U7-BST): track 0.00 -> 2.23 mm
- net Net-(D6-A): track 0.00 -> 2.01 mm
- net Net-(R20-Pad2): track 0.00 -> 2.00 mm
- net GND: vias 0 -> 22
- added copper zone on F.Cu, net +5V
- added copper zone on B.Cu, net /VBAT
- added copper zone on F.Cu, net /VBAT
- added copper zone on In2.Cu, net /VBAT
- added copper zone on In1.Cu, net GND
- added copper zone on F.Cu, net Net-(D5-K)
- added copper zone on F.Cu, net Net-(U7-SW)
Other:
- outline, holes or cut-outs redrawn
- copper layers 2 -> 4

Commit message: Se corrigio pcb y se agrego conectores molex a sensores
Parts:
- added J2: Conn_01x03, Connector_Molex:Molex_KK-254_AE-6410-03A_1x03_P2.54mm_Vertical, F.Cu at (100.7, 140.1)
- added J4: Conn_01x02, Connector_Molex:Molex_KK-254_AE-6410-02A_1x02_P2.54mm_Vertical, F.Cu at (108.5, 139.9)
- added J6: Conn_01x04, Connector_Molex:Molex_KK-254_AE-6410-04A_1x04_P2.54mm_Vertical, F.Cu at (93.1, 140.1)
- U5: moved to F.Cu
- moved Y1 226.5 mm to (46.6, 123.5), turned to 90 degrees
- moved U1 222.9 mm to (58.4, 125.0)
- moved C2 212.6 mm to (49.4, 125.5), turned to -90 degrees
- moved C3 211.9 mm to (49.4, 121.7), turned to 90 degrees
- moved C8 209.3 mm to (51.4, 127.4), turned to -90 degrees
- moved C9 208.3 mm to (52.1, 120.3), turned to 90 degrees
- moved C5 205.3 mm to (55.3, 117.6)
- moved C7 198.7 mm to (62.6, 131.6), turned to 180 degrees
- moved C6 194.4 mm to (66.3, 121.9), turned to -90 degrees
- moved R13 144.8 mm to (127.1, 197.8)
- moved J1 143.0 mm to (125.1, 113.8), turned to 90 degrees
- moved U2 85.3 mm to (182.6, 110.6)
- moved D6 23.3 mm to (149.8, 138.5), turned to -90 degrees
- moved R18 18.8 mm to (152.2, 139.0), turned to -90 degrees
- moved C15 15.1 mm to (123.5, 130.0), turned to 90 degrees
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Connections:
- J10 pad 1: /MOTOR/MOTA_R -> /MOTOR/MOTB_R
- J10 pad 2: /MOTOR/MOTB_R -> /MOTOR/MOTA_R
- J11 pad 1: /MOTOR/MOTB_L -> /MOTOR/MOTA_L
- J11 pad 2: /MOTOR/MOTA_L -> /MOTOR/MOTB_L
Routing:
- net GND: track 0.00 -> 42.7 mm, vias 22 -> 32
- net +3.3V: track 0.00 -> 34.5 mm, vias 0 -> 4
- net +5V: track 2.44 -> 13.5 mm, vias 10 -> 6
- net /OSC_A: track 0.00 -> 10.4 mm
- net /VBAT: track 4.25 -> 14.3 mm, vias 29 -> 39
- net Net-(D5-A): track 9.52 -> 17.3 mm, vias 3 -> 0
- net /OSC_B: track 0.00 -> 6.85 mm
- net /MOTOR/MODE_ML: track 0.00 -> 4.75 mm, vias 0 -> 1
- net /MOTOR/MODE_MR: track 0.00 -> 4.53 mm, vias 0 -> 1
- net Net-(U7-EN): track 2.74 -> 7.20 mm
- net Net-(D5-K): track 4.01 -> 0.00 mm, vias 0 -> 10
- net Net-(U7-SW): track 3.87 -> 0.00 mm
- net Net-(SW6-A): track 3.06 -> 5.08 mm
- net Net-(U7-FB): track 9.61 -> 9.30 mm, vias 2 -> 0
- added copper zone on In2.Cu, net +5V
- added copper zone on F.Cu, net /MOTOR/MOTA_L
- added copper zone on F.Cu, net /MOTOR/MOTA_R
- added copper zone on F.Cu, net /MOTOR/MOTB_L
- added copper zone on F.Cu, net /MOTOR/MOTB_R
- added copper zone on F.Cu, net GND
- added copper zone on In2.Cu, net Net-(D5-K)
- removed copper zone on B.Cu, net /VBAT

Commit message: Se ruteo y se cambio conectores a jst ph 2mm
Parts:
- added C24: 100nF, Capacitor_SMD:C_0603_1608Metric, F.Cu at (150.7, 116.4)
- added C25: 100nF, Capacitor_SMD:C_0603_1608Metric, F.Cu at (146.9, 119.3)
- added U12: AP2112K-3.3TRG1, Package_TO_SOT_SMD:SOT-23-5, F.Cu at (150.3, 119.3)
- added kibuzzard-6A769CB5: G***, kibuzzard-6A769CB5, F.Cu at (102.0, 115.0)
- added kibuzzard-6A769EC5: G***, kibuzzard-6A769EC5, F.Cu at (99.0, 116.0)
- added kibuzzard-6A769EE0: G***, kibuzzard-6A769EE0, F.Cu at (96.0, 114.0)
- added kibuzzard-6A769EE9: G***, kibuzzard-6A769EE9, F.Cu at (93.0, 114.0)
- C20, C21: value 22uF -> 100nF
- J2: footprint Connector_Molex:Molex_KK-254_AE-6410-03A_1x03_P2.54mm_Vertical -> Connector_JST:JST_PH_S3B-PH-K_1x03_P2.00mm_Horizontal; moved to B.Cu
- J3: footprint Connector_PinHeader_2.54mm:PinHeader_1x03_P2.54mm_Vertical -> Connector_PinHeader_2.54mm:PinHeader_1x03_P2.54mm_Horizontal; moved to B.Cu
- J4: footprint Connector_Molex:Molex_KK-254_AE-6410-02A_1x02_P2.54mm_Vertical -> Connector_JST:JST_PH_S2B-PH-K_1x02_P2.00mm_Horizontal; moved to B.Cu
- J6: footprint Connector_Molex:Molex_KK-254_AE-6410-04A_1x04_P2.54mm_Vertical -> Connector_JST:JST_PH_S4B-PH-K_1x04_P2.00mm_Horizontal; moved to B.Cu
- moved D1 186.7 mm to (93.0, 110.0), turned to 90 degrees
- moved D2 183.8 mm to (96.0, 110.0), turned to 90 degrees
- moved D3 181.0 mm to (99.0, 110.0), turned to 90 degrees
- moved R9 180.5 mm to (89.0, 117.0), turned to 90 degrees
- moved R5 179.8 mm to (85.0, 117.0), turned to 90 degrees
- moved R10 178.6 mm to (91.0, 117.0), turned to 90 degrees
- moved D4 178.2 mm to (102.0, 110.0), turned to 90 degrees
- moved R6 177.8 mm to (87.0, 117.0), turned to 90 degrees
- moved R3 155.6 mm to (110.2, 133.0), turned to 180 degrees
- moved R4 155.6 mm to (110.2, 135.5)
- moved C11 151.8 mm to (124.7, 110.5)
- moved R15 150.1 mm to (124.5, 112.5)
- moved C10 147.6 mm to (129.0, 112.7), turned to 180 degrees
- moved R14 145.5 mm to (129.1, 110.6), turned to 180 degrees
- moved C4 128.7 mm to (132.5, 118.8), turned to -90 degrees
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Connections:
- D1 pad 1: GND -> Net-(D1-K)
- D1 pad 2: Net-(D1-A) -> +3.3V
- D2 pad 1: GND -> Net-(D2-K)
- D2 pad 2: Net-(D2-A) -> +3.3V
- D3 pad 1: GND -> Net-(D3-K)
- D3 pad 2: Net-(D3-A) -> +3.3V
- D4 pad 1: GND -> Net-(D4-K)
- D4 pad 2: Net-(D4-A) -> +3.3V
- J4 pad 1: GND -> +3V3
- J4 pad 2: +3.3V -> GND
- R10 pad 2: Net-(D4-A) -> Net-(D4-K)
- R5 pad 2: Net-(D1-A) -> Net-(D1-K)
- R6 pad 2: Net-(D2-A) -> Net-(D2-K)
- R9 pad 2: Net-(D3-A) -> Net-(D3-K)
- U1 pad 2: /LED2 -> /LED3
- U1 pad 29: /PWMB_MOTR -> /PWMA_MOTL
- U1 pad 3: /LED3 -> /LED2
- U1 pad 30: /PWMA_MOTR -> /PWMB_MOTL
- U1 pad 31: /PWMB_MOTL -> /PWMA_MOTR
- U1 pad 32: /PWMA_MOTL -> /PWMB_MOTR
- U1 pad 4: /LED4 -> /LED1
- U1 pad 46: /LED1 -> /LED4
Routing:
- net /NRST: track 0.00 -> 73.7 mm, vias 0 -> 2
- net +3.3V: track 34.5 -> 89.7 mm, vias 4 -> 13
- net /BOOT0: track 0.00 -> 46.5 mm, vias 0 -> 2
- net /PWMB_MOTR: track 0.00 -> 44.5 mm
- net /PWMA_MOTR: track 0.00 -> 43.8 mm
- net GND: track 42.7 -> 78.6 mm, vias 32 -> 41
- net /IR_38khz: track 0.00 -> 35.8 mm, vias 0 -> 1
- net /SWCLK: track 0.00 -> 28.5 mm
- net /SWDIO: track 0.00 -> 27.0 mm
- net +5V: track 13.5 -> 39.3 mm, vias 6 -> 12
- net /PWMB_MOTL: track 0.00 -> 24.9 mm
- net /PWMA_MOTL: track 0.00 -> 23.8 mm
- net /VOLTAGE: track 0.00 -> 20.7 mm
- net /Linea3: track 0.00 -> 19.8 mm, vias 0 -> 1
- net /Linea2: track 0.00 -> 18.5 mm, vias 0 -> 1
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- added copper zone on In2.Cu, net +3.3V
- added copper zone on In2.Cu, net +3V3
