File: Inda_Kidcad/Inda_Kidcad.kicad_pcb (KiCad board)
At the start: 4 copper layers, 88 x 55.2 mm, 104 parts, among them J1 SWD_UART_CONN, J10 CONN_MR, J11 CONN_ML, J12 XT30, J13 Conn_01x03_Pin, J14 Conn_01x03_Pin, J15 Conn_01x03_Pin, J2 Conn_01x03, J3 Conn_01x03, J4 Conn_01x02, J5 SQJ951EP, J6 Conn_01x04, SW1 SW_Push, SW2 SW_Push, SW3 SW_Push, SW4 SW_Push, SW5 SW_Push, SW6 SW_Push_SPDT, U1 STM32f103C8t6, U10 QRE111GR, U12 AP2112K-3.3TRG1, U2 vs1838, U3 DRV8212DSGR, U4 DRV8212DSGR, U6 AP2112K-3.3TRG1, U7 MSTPS563200DDCR, U8 QRE111GR, U9 QRE111GR, Y1 8Mhz

Commit message: rev 2.0 con 4 capas y terminada a falta de revision
Parts:
- removed kibuzzard-6A769EE0: G***, kibuzzard-6A769EE0
- removed kibuzzard-6A769EE9: G***, kibuzzard-6A769EE9
- added G***: LOGO, LOGO, B.Cu at (93.5, 118.5)
- added kibuzzard-6A7EB2CB: G***, kibuzzard-6A7EB2CB, F.Cu at (96.0, 115.3)
- added kibuzzard-6A824811: G***, kibuzzard-6A824811, F.Cu at (93.0, 115.0)
- added kibuzzard-6A824831: G***, kibuzzard-6A824831, F.Cu at (118.9, 126.0)
- added kibuzzard-6A824876: G***, kibuzzard-6A824876, F.Cu at (127.0, 126.0)
- added kibuzzard-6A824881: G***, kibuzzard-6A824881, F.Cu at (111.0, 126.0)
- added kibuzzard-6A824B6A: G***, kibuzzard-6A824B6A, F.Cu at (146.0, 109.8)
- added kibuzzard-6A824B7E: G***, kibuzzard-6A824B7E, F.Cu at (147.0, 114.2)
- added kibuzzard-6A824C7C: G***, kibuzzard-6A824C7C, B.Cu at (149.5, 133.0)
- added kibuzzard-6A824CA2: G***, kibuzzard-6A824CA2, B.Cu at (150.2, 127.0)
- added kibuzzard-6A824CC5: G***, kibuzzard-6A824CC5, B.Cu at (145.5, 118.5)
- added kibuzzard-6A824CCF: G***, kibuzzard-6A824CCF, B.Cu at (145.2, 121.0)
- added kibuzzard-6A824CD8: G***, kibuzzard-6A824CD8, B.Cu at (146.2, 123.5)
- added kibuzzard-6A824CFB: G***, kibuzzard-6A824CFB, B.Cu at (156.2, 111.5)
- added kibuzzard-6A824D03: G***, kibuzzard-6A824D03, B.Cu at (156.5, 113.5)
- added kibuzzard-6A824D25: G***, kibuzzard-6A824D25, B.Cu at (92.5, 131.0)
- added kibuzzard-6A824D2A: G***, kibuzzard-6A824D2A, B.Cu at (94.5, 131.0)
- added kibuzzard-6A824D2F: G***, kibuzzard-6A824D2F, B.Cu at (96.5, 131.0)
- added kibuzzard-6A824D39: G***, kibuzzard-6A824D39, B.Cu at (105.5, 131.2)
- added kibuzzard-6A824D40: G***, kibuzzard-6A824D40, B.Cu at (98.5, 131.0)
- added kibuzzard-6A824D46: G***, kibuzzard-6A824D46, B.Cu at (107.5, 131.2)
- added kibuzzard-6A824D4A: G***, kibuzzard-6A824D4A, B.Cu at (109.5, 131.2)
- added kibuzzard-6A824E30: G***, kibuzzard-6A824E30, B.Cu at (155.0, 101.5)
- added kibuzzard-6A824E30: G***, kibuzzard-6A824E30, B.Cu at (115.0, 101.2)
- added kibuzzard-6A824E30: G***, kibuzzard-6A824E30, B.Cu at (139.8, 128.5)
- added kibuzzard-6A824E30: G***, kibuzzard-6A824E30, B.Cu at (135.0, 101.2)
- added kibuzzard-6A824E30: G***, kibuzzard-6A824E30, B.Cu at (127.8, 128.5)
- added kibuzzard-6A824E39: G***, kibuzzard-6A824E39, B.Cu at (127.2, 131.2)
- added kibuzzard-6A824E39: G***, kibuzzard-6A824E39, B.Cu at (157.2, 102.0)
- added kibuzzard-6A824E39: G***, kibuzzard-6A824E39, B.Cu at (137.2, 101.8)
- added kibuzzard-6A824E39: G***, kibuzzard-6A824E39, B.Cu at (140.0, 131.5)
- added kibuzzard-6A824E39: G***, kibuzzard-6A824E39, B.Cu at (117.2, 101.8)
- added kibuzzard-6A824EDE: G***, kibuzzard-6A824EDE, B.Cu at (152.8, 102.0)
- added kibuzzard-6A824EDE: G***, kibuzzard-6A824EDE, B.Cu at (132.8, 101.8)
- added kibuzzard-6A824EDE: G***, kibuzzard-6A824EDE, B.Cu at (112.8, 101.8)
- added kibuzzard-6A8256E6: G***, kibuzzard-6A8256E6, B.Cu at (93.0, 109.0)
- R22, R23, R24, R25, R26, R27: footprint Resistor_SMD:R_0805_2012Metric_Pad1.20x1.40mm_HandSolder -> Resistor_SMD:R_0603_1608Metric
- SW3, SW4, SW5: footprint Button_Switch_SMD:SW_SPST_CK_RS282G05A3 -> Button_Switch_SMD:SW_Push_SPST_NO_Alps_SKRK
- moved J13 203.2 mm to (115.0, 102.8)
- moved C26 201.6 mm to (115.8, 99.5)
- moved U8 196.2 mm to (115.0, 96.0), turned to 180 degrees
- moved R23 194.3 mm to (111.0, 98.0), turned to 90 degrees
- moved R22 186.1 mm to (119.0, 98.1), turned to 90 degrees
- moved J14 183.4 mm to (135.0, 102.8)
- moved C27 182.2 mm to (135.5, 99.5)
- moved U9 176.5 mm to (135.0, 96.0), turned to 180 degrees
- moved R25 174.5 mm to (131.2, 98.1), turned to 90 degrees
- moved R7 170.0 mm to (111.0, 123.5)
- moved R8 169.8 mm to (110.2, 130.6)
- moved R12 168.7 mm to (118.0, 123.0)
- moved R24 166.5 mm to (139.0, 98.1), turned to 90 degrees
- moved J15 163.7 mm to (155.0, 102.8)
- moved C28 162.5 mm to (155.8, 99.5)
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Routing:
- net +3.3V: track 89.7 -> 172.4 mm, vias 13 -> 21
- net /SELECTOR: track 0.00 -> 63.1 mm, vias 0 -> 6
- net /SERVO: track 0.00 -> 51.9 mm, vias 0 -> 1
- net /TX: track 0.00 -> 29.7 mm, vias 0 -> 2
- net /RX: track 0.00 -> 26.2 mm, vias 0 -> 2
- net GND: track 78.6 -> 92.3 mm, vias 41 -> 119
- net /SENSOR_LINEA/CONN1_3V3: track 0.00 -> 12.4 mm
- net /SENSOR_LINEA/CONN2_3V3: track 0.00 -> 12.2 mm
- net /SENSOR_LINEA/CONN3_3V3: track 0.00 -> 11.6 mm
- net /SENSOR_LINEA/CONN_IR3: track 0.00 -> 8.04 mm, vias 0 -> 2
- net /SENSOR_LINEA/CONN_IR1: track 0.00 -> 7.82 mm, vias 0 -> 2
- net /SENSOR_LINEA/CONN_IR2: track 0.00 -> 7.77 mm, vias 0 -> 2
- net /SENSOR_LINEA/CONN3_GND: track 0.00 -> 7.62 mm, vias 0 -> 7
- net /SENSOR_LINEA/CONN2_GND: track 0.00 -> 7.06 mm, vias 0 -> 7
- net /SENSOR_LINEA/CONN1_GND: track 0.00 -> 6.65 mm, vias 0 -> 7
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- added copper zone on B.Cu, net /SENSOR_LINEA/CONN1_GND
- added copper zone on F.Cu, net /SENSOR_LINEA/CONN1_GND
- added copper zone on In1.Cu, net /SENSOR_LINEA/CONN1_GND
- added copper zone on In2.Cu, net /SENSOR_LINEA/CONN1_GND
- added copper zone on B.Cu, net /SENSOR_LINEA/CONN2_GND
- added copper zone on F.Cu, net /SENSOR_LINEA/CONN2_GND
- added copper zone on In1.Cu, net /SENSOR_LINEA/CONN2_GND
- added copper zone on In2.Cu, net /SENSOR_LINEA/CONN2_GND
- added copper zone on B.Cu, net /SENSOR_LINEA/CONN3_GND
- added copper zone on F.Cu, net /SENSOR_LINEA/CONN3_GND
- added copper zone on In1.Cu, net /SENSOR_LINEA/CONN3_GND
- added copper zone on In2.Cu, net /SENSOR_LINEA/CONN3_GND
- added copper zone on B.Cu, net GND
- added copper zone on In2.Cu, net GND
Other:
- board size 88 x 55.2 mm -> 88 x 48.5 mm

Commit message: Terminado mini sumo v2 a espera de revision
Parts:
- J12: footprint Footprint:XT30_H_M -> Connector_AMASS:AMASS_XT30PW-M_1x02_P2.50mm_Horizontal
- moved J12 2.50 mm to (167.5, 133.0), turned to -90 degrees
Connections:
- U1 pad 18: /Mod_TX2 -> unconnected-(U1-PB0_ADC8_PWM3-Pad18)
- U1 pad 19: /Mod_TX3 -> unconnected-(U1-PB1_ADC9_PWM3-Pad19)
Routing:
- net Net-(D5-A): track 17.3 -> 19.4 mm, vias 0 -> 2
- net /VBAT: vias 40 -> 39
