File: Inda_Kidcad/Inda_Kidcad.kicad_pcb (KiCad board)
At the start: 4 copper layers, 88 x 48.5 mm, 138 parts, among them J1 SWD_UART_CONN, J10 CONN_MR, J11 CONN_ML, J12 XT30, J13 Conn_01x03_Pin, J14 Conn_01x03_Pin, J15 Conn_01x03_Pin, J2 Conn_01x03, J3 Conn_01x03, J4 Conn_01x02, J5 SQJ951EP, J6 Conn_01x04, SW1 SW_Push, SW2 SW_Push, SW3 SW_Push, SW4 SW_Push, SW5 SW_Push, SW6 SW_Push_SPDT, U1 STM32f103C8t6, U10 QRE111GR, U12 AP2112K-3.3TRG1, U2 vs1838, U3 DRV8212DSGR, U4 DRV8212DSGR, U6 AP2112K-3.3TRG1, U7 MSTPS563200DDCR, U8 QRE111GR, U9 QRE111GR, Y1 8Mhz

Commit message: cambios ultimos
Parts:
- added R29: 100K, Resistor_SMD:R_0603_1608Metric_Pad0.98x0.95mm_HandSolder, F.Cu at (164.6, 134.5)
- R1, R13, R2: footprint Capacitor_SMD:C_0805_2012Metric_Pad1.18x1.45mm_HandSolder -> Resistor_SMD:R_0603_1608Metric_Pad0.98x0.95mm_HandSolder
- R10, R11, R12, R14, R15, R18, R3, R4, R5, R6, R7, R8, R9: footprint Resistor_SMD:R_0805_2012Metric_Pad1.20x1.40mm_HandSolder -> Resistor_SMD:R_0603_1608Metric_Pad0.98x0.95mm_HandSolder
- R17: value 100K -> 1k; footprint Resistor_SMD:R_0805_2012Metric_Pad1.20x1.40mm_HandSolder -> Resistor_SMD:R_0603_1608Metric_Pad0.98x0.95mm_HandSolder
- R22, R23, R24, R25, R26, R27: footprint Resistor_SMD:R_0603_1608Metric -> Resistor_SMD:R_0603_1608Metric_Pad0.98x0.95mm_HandSolder
- moved D5 0.50 mm to (162.5, 133.8)
Routing:
- net Net-(D5-K): track 0.00 -> 2.67 mm
- net Net-(D5-A): track 19.4 -> 21.6 mm
Other:
- outline, holes or cut-outs redrawn
- board text added: "+"
