File: Inda_Kidcad/ALIMENTACION.kicad_sch (KiCad schematic)
At the start: 15 parts, among them U6 CN3903, U7 AMS1117-5.0

Commit message: Version 2 De Sumo Inda
Parts:
- removed C24, C25, C27: 100nF, Capacitor_SMD:C_0603_1608Metric, symbol Device:C
- removed C26: 22uF, Capacitor_SMD:C_0603_1608Metric, symbol Device:C
- removed C28: 10uF, Capacitor_SMD:CP_Elec_4x5.8, symbol Device:C_Polarized
- removed C29, C30: 10uF, Capacitor_SMD:C_1206_3216Metric_Pad1.33x1.80mm_HandSolder, symbol Device:C_Polarized
- removed L5: 4.7uH, Inductor_SMD:L_Wuerth_HCM-7050, symbol Device:L
- removed U6: CN3903, Package_SO:HSOP-8-1EP_3.9x4.9mm_P1.27mm_EP2.41x3.1mm, symbol Micromouse_Library:CN3903
- removed U7: AMS1117-5.0, Package_TO_SOT_SMD:SOT-223-3_TabPin2, symbol Regulator_Linear:AMS1117-5.0
- added C36, C40, C41, C42, C43: 22uF, Capacitor_SMD:C_0603_1608Metric, symbol Device:C
- added C39: 0.1uF, Capacitor_SMD:C_0603_1608Metric, symbol Device:C
- added D5: 12V, Resistor_SMD:R_1206_3216Metric_Pad1.30x1.75mm_HandSolder, symbol Device:D_Zener
- added D6: GREEN, LED_SMD:LED_1206_3216Metric_Pad1.42x1.75mm_HandSolder, symbol Device:LED
- added J3: BRIDGE, Connector_PinHeader_2.54mm:PinHeader_1x02_P2.54mm_Vertical, symbol Connector:Conn_01x02_Pin
- added J7: XT30, Connector_AMASS:AMASS_XT30U-F_1x02_P5.0mm_Vertical, symbol LIB_CONECTORES:Conector_XT30
- added L1: 3.3uH, symbol Device:L
- added Q5, Q6: AO3401A, Package_TO_SOT_SMD:SOT-23, symbol Transistor_FET:AO3401A
- added R18, R19: 100K, Resistor_SMD:R_0805_2012Metric_Pad1.20x1.40mm_HandSolder, symbol Device:R
- added R20: 20K, Resistor_SMD:R_0805_2012Metric_Pad1.20x1.40mm_HandSolder, symbol Device:R
- added SW3: SW_Push_SPDT, Button_Switch_SMD:SW_SPDT_PCM12, symbol Switch:SW_Push_SPDT
- added U3: AP2112K-3.3TRG1, Package_TO_SOT_SMD:SOT-23-5, symbol LIB_REGULADORES:AP2112K-3.3TRG1
- added U4: MSTPS563200DDCR, Package_TO_SOT_SMD:SOT-23-6, symbol LIB_REGULADORES:MSTPS563200DDCR_BUCK
- R21: value 18k -> 200K; footprint Resistor_SMD:R_0805_2012Metric_Pad1.20x1.40mm_HandSolder -> Resistor_SMD:R_0603_1608Metric_Pad0.98x0.95mm_HandSolder
- R22: value 100K -> 116K; footprint Resistor_SMD:R_0805_2012Metric_Pad1.20x1.40mm_HandSolder -> Resistor_SMD:R_0603_1608Metric_Pad0.98x0.95mm_HandSolder
- R23: value 39k -> 22K; footprint Resistor_SMD:R_0805_2012Metric_Pad1.20x1.40mm_HandSolder -> Resistor_SMD:R_0603_1608Metric_Pad0.98x0.95mm_HandSolder
Connections:
- net +3.3V: now also C43.2, U3.5 (VOUT); no longer R22.2
- net +5V: now also R22.1, C40.2, C41.2, C42.2, L1.1, U3.1 (VIN), U3.3 (EN)
- net GND: now also R23.2, C36.1, C40.1, C41.1, C42.1, C43.1, D6.1 (K), J7.1 (GND), SW3.2 (B), U3.2 (GND), U4.1 (GND); no longer R23.1
- net VBAT: now reaches R21.2
- net VBAT: now also C31.1, C32.2, J3.1 (Pin_1), Q6.3 (D), R20.1
- removed net FB: R22.1, R23.2
- removed net VIN: C31.1, C32.2, R21.1
- new net: J3.2 (Pin_2), J7.2 (VCC), Q5.3 (D)
- new net: D5.2 (A), Q5.1 (G), Q6.1 (G), R19.1
- new net: D5.1 (K), Q5.2 (S), Q6.2 (S), R18.1
- new net: D6.2 (A), R20.2
- new net: R18.2, R19.2, SW3.1 (A)
- new net: R22.2, R23.1, U4.4 (FB)
- new net: C39.1, U4.6 (BST)
- new net: C39.2, L1.2, U4.2 (SW)
- new net: R21.1, U4.5 (EN)
- new net: C36.2, U4.3 (VIN)
- no-connect marks 0 -> 2
Other:
- moved on the sheet: C31, C32

Commit message: Se cambia simbolos como huellas, se coloca solo mosfet para interruptor y se empieza con pcb
Parts:
- removed C36, C40, C41: 22uF, Capacitor_SMD:C_0603_1608Metric, symbol Device:C
- removed J3: BRIDGE, Connector_PinHeader_2.54mm:PinHeader_1x02_P2.54mm_Vertical, symbol Connector:Conn_01x02_Pin
- removed Q5, Q6: AO3401A, Package_TO_SOT_SMD:SOT-23, symbol Transistor_FET:AO3401A
- removed R18: 100K, Resistor_SMD:R_0805_2012Metric_Pad1.20x1.40mm_HandSolder, symbol Device:R
- added C23: 22uF, Capacitor_SMD:C_0603_1608Metric, symbol Device:C
- added C29, C30: 22uF, Capacitor_Tantalum_SMD:CP_EIA-3528-15_AVX-H_HandSolder, symbol Device:C_Polarized
- added J5: SQJ951EP, Package_SO:PowerPAK_SO-8_Dual, symbol LIB_MOSFET_BJT:SQJ951EP-T1_BE3
- added R28: 15k, Resistor_SMD:R_0603_1608Metric_Pad0.98x0.95mm_HandSolder, symbol Device:R
- added U5: (no value), Footprint:BRIDGE_2P, symbol LIB_CONECTORES:BRIDGE_2P
- J12: renamed from J7; footprint Connector_AMASS:AMASS_XT30U-F_1x02_P5.0mm_Vertical -> Footprint:XT30_H_M
- L1: footprint (none) -> Inductor_SMD:L_Sunlord_MWSA0402S
- R18: renamed from R20; value 20K -> 10k
- R20: renamed from R22; value 116K -> 100k
- renumbered C31 to C18, C32 to C19, C42 to C20, C43 to C21, C39 to C22, R19 to R17, R21 to R19, R23 to R21, SW3 to SW6, U3 to U6, U4 to U7
Connections:
- net +5V: now also C23.2, C30.1
- net GND: now also C23.1, C29.2, C30.2
- net VBAT: now also U7.3 (VIN), C29.1, J5.5 (D1), J5.6 (D2), U5.2 (B)
- net at J12.2 (VCC): now also D5.1 (K), J5.1 (S1), J5.3 (S2), U5.1 (A)
- net at D5.2 (A), R17.1: now also J5.2 (G1), J5.4 (G2)
- net at R21.1, U7.4 (FB): now also R28.2; no longer R20.2
- new net: R20.2, R28.1
Other:
- moved on the sheet: C18, C19, C20, C21, C22, D5, D6, J12, L1, R17, R18, R19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

Commit message: Se ruteo y se cambio conectores a jst ph 2mm
Parts:
- added C24, C25: 100nF, Capacitor_SMD:C_0603_1608Metric, symbol Device:C
- added U12: AP2112K-3.3TRG1, Package_TO_SOT_SMD:SOT-23-5, symbol LIB_REGULADORES:AP2112K-3.3TRG1
- C20, C21: value 22uF -> 100nF
Connections:
- net +5V: now also C24.2, U12.1 (VIN), U12.3 (EN)
- net GND: now also C24.1, C25.1, U12.2 (GND)
- new net +3V3: C25.2, U12.5 (VOUT)
- no-connect marks 2 -> 3

Commit message: Terminado mini sumo v2 a espera de revision
Parts:
- J12: footprint Footprint:XT30_H_M -> Connector_AMASS:AMASS_XT30PW-M_1x02_P2.50mm_Horizontal
Changed lines of the file:
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@@
 			)
 		)
-		(property "Footprint" "Footprint:XT30_H_M"
+		(property "Footprint" "Connector_AMASS:AMASS_XT30PW-M_1x02_P2.50mm_Horizontal"
 			(at 17.78 35.56 0)
 			(hide yes)

Commit message: cambios ultimos
Parts:
- added R29: 100K, Resistor_SMD:R_0603_1608Metric_Pad0.98x0.95mm_HandSolder, symbol Device:R
- R17: value 100K -> 1k; footprint Resistor_SMD:R_0805_2012Metric_Pad1.20x1.40mm_HandSolder -> Resistor_SMD:R_0603_1608Metric_Pad0.98x0.95mm_HandSolder
- R18: footprint Resistor_SMD:R_0805_2012Metric_Pad1.20x1.40mm_HandSolder -> Resistor_SMD:R_0603_1608Metric_Pad0.98x0.95mm_HandSolder
Connections:
- net at D5.1 (K), J12.2 (VCC), J5.1 (S1)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: now also R29.1
- net at D5.2 (A), J5.2 (G1), J5.4 (G2)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: now also R29.2
Other:
- moved on the sheet: J12
Changed lines of the file:
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@@
 	)
 	(junction
+		(at 38.1 16.51)
+		(diameter 0)
+		(color 0 0 0 0)
+	)
+	(junction
 		(at 24.13 76.2)
 		(diameter 0)
@@
 	)
 	(junction
-		(at 38.1 15.24)
-		(diameter 0)
-		(color 0 0 0 0)
-	)
-	(junction
 		(at 38.1 45.72)
 		(diameter 0)
@@
 		(color 0 0 0 0)
 	)
+	(junction
+		(at 30.48 16.51)
+		(diameter 0)
+		(color 0 0 0 0)
+	)
 	(no_connect
 		(at 62.23 168.91)
@@
 	(wire
 		(pts
-			(xy 33.02 15.24) (xy 33.02 31.75)
+			(xy 25.4 16.51) (xy 25.4 31.75)
+		)
+		(stroke
+			(width 0)
+			(type default)
+		)
+	)
+	(wire
+		(pts
+			(xy 24.13 31.75) (xy 25.4 31.75)
 		)
 		(stroke
@@
 	(wire
 		(pts
+			(xy 30.48 16.51) (xy 38.1 16.51)
+		)
+		(stroke
+			(width 0)
+			(type default)
+		)
+	)
+	(wire
+		(pts
 			(xy 45.72 31.75) (xy 45.72 21.59)
 		)
@@
 	(wire
 		(pts
-			(xy 29.21 34.29) (xy 33.02 34.29)
+			(xy 24.13 34.29) (xy 25.4 34.29)
 		)
 		(stroke
@@
 	(wire
 		(pts
+			(xy 30.48 35.56) (xy 30.48 45.72)
+		)
+		(stroke
+			(width 0)
+			(type default)
+		)
+	)
+	(wire
+		(pts
 			(xy 157.48 55.88) (xy 157.48 59.69)
 		)
@@
 	(wire
 		(pts
+			(xy 30.48 16.51) (xy 30.48 27.94)
+		)
+		(stroke
+			(width 0)
+			(type default)
+		)
+	)
+	(wire
+		(pts
 			(xy 71.12 104.14) (xy 71.12 107.95)
 		)
@@
 	(wire
 		(pts
+			(xy 38.1 16.51) (xy 38.1 15.24)
+		)
+		(stroke
+			(width 0)
+			(type default)
+		)
+	)
+	(wire
+		(pts
 			(xy 68.58 157.48) (xy 68.58 161.29)
 		)
@@
 	(wire
 		(pts
-			(xy 29.21 31.75) (xy 33.02 31.75)
+			(xy 182.88 73.66) (xy 182.88 77.47)
 		)
 		(stroke
@@
 	(wire
 		(pts
-			(xy 182.88 73.66) (xy 182.88 77.47)
+			(xy 30.48 45.72) (xy 38.1 45.72)
 		)
 		(stroke
@@
 	(wire
 		(pts
-			(xy 33.02 34.29) (xy 33.02 38.1)
+			(xy 25.4 34.29) (xy 25.4 38.1)
 		)
 		(stroke
@@
 	(wire
 		(pts
-			(xy 33.02 15.24) (xy 38.1 15.24)
+			(xy 25.4 16.51) (xy 30.48 16.51)
 		)
 		(stroke
@@
 	(wire
 		(pts
-			(xy 38.1 21.59) (xy 38.1 15.24)
+			(xy 38.1 21.59) (xy 38.1 16.51)
 		)
 		(stroke
@@
 	(symbol
 		(lib_id "LIB_CONECTORES:Conector_XT30")
-		(at 17.78 35.56 0)
+		(at 12.7 35.56 0)
 		(mirror x)
 		(unit 1)
@@
 		(dnp no)
 		(property "Reference" "J12"
-			(at 25.146 27.686 0)
+			(at 20.066 27.686 0)
 			(show_name no)
 			(do_not_autoplace no)
@@
 		)
 		(property "Value" "XT30"
-			(at 17.272 27.94 0)
+			(at 12.192 27.94 0)
 			(show_name no)
 			(do_not_autoplace no)
@@
 		)
 		(property "Footprint" "Connector_AMASS:AMASS_XT30PW-M_1x02_P2.50mm_Horizontal"
-			(at 17.78 35.56 0)
+			(at 12.7 35.56 0)
 			(hide yes)
 			(show_name no)
@@
 		)
 		(property "Datasheet" ""
-			(at 17.78 35.56 0)
+			(at 12.7 35.56 0)
 			(hide yes)
 			(show_name no)
@@
 		)
 		(property "Description" ""
-			(at 17.78 35.56 0)
+			(at 12.7 35.56 0)
 			(hide yes)
 			(show_name no)
@@
 	)
 	(symbol
+		(lib_id "Device:R")
+		(at 30.48 31.75 0)
+		(unit 1)
+		(body_style 1)
+		(exclude_from_sim no)
+		(in_bom yes)
+		(on_board yes)
+		(in_pos_files yes)
+		(dnp no)
+		(fields_autoplaced yes)
+		(property "Reference" "R29"
+			(at 33.02 30.4799 0)
+			(show_name no)
+			(do_not_autoplace no)
+			(effects
+				(font
+					(size 1.27 1.27)
+				)
+				(justify left)
+			)
+		)
+		(property "Value" "100K"
+			(at 33.02 33.0199 0)
+			(show_name no)
+			(do_not_autoplace no)
+			(effects
+				(font
+					(size 1.27 1.27)
+				)
+				(justify left)
+			)
+		)
+		(property "Footprint" "Resistor_SMD:R_0603_1608Metric_Pad0.98x0.95mm_HandSolder"
+			(at 28.702 31.75 90)
+			(hide yes)
+			(show_name no)
+			(do_not_autoplace no)
+			(effects
+				(font
+					(size 1.27 1.27)
+				)
+			)
+		)
+		(property "Datasheet" ""
+			(at 30.48 31.75 0)
+			(hide yes)
+			(show_name no)
+			(do_not_autoplace no)
+			(effects
+				(font
+					(size 1.27 1.27)
+				)
+			)
+		)
+		(property "Description" "Resistor"
+			(at 30.48 31.75 0)
+			(hide yes)
+			(show_name no)
+			(do_not_autoplace no)
+			(effects
+				(font
+					(size 1.27 1.27)
+				)
+			)
+		)
+		(pin "2"
+		)
+		(pin "1"
+		)
+		(instances
+			(project "Inda_Kidcad"
+				(path "/0fd92b06-954d-41bf-a53b-1bc8635b69f8/b022e595-33bd-440b-84f6-8dfa037dfa4f"
+					(reference "R29")
+					(unit 1)
+				)
+			)
+		)
+	)
+	(symbol
 		(lib_id "power:+5V")
 		(at 30.48 105.41 0)
@@
 	(symbol
 		(lib_id "power:GND")
-		(at 33.02 38.1 0)
+		(at 25.4 38.1 0)
 		(unit 1)
 		(body_style 1)
@@
 		(fields_autoplaced yes)
 		(property "Reference" "#PWR053"
-			(at 33.02 44.45 0)
+			(at 25.4 44.45 0)
 			(hide yes)
 			(show_name no)
@@
 		)
 		(property "Value" "GND"
-			(at 33.02 43.18 0)
+			(at 25.4 43.18 0)
 			(show_name no)
 			(do_not_autoplace no)
@@
 		)
 		(property "Footprint" ""
-			(at 33.02 38.1 0)
+			(at 25.4 38.1 0)
 			(hide yes)
 			(show_name no)
@@
 		)
 		(property "Datasheet" ""
-			(at 33.02 38.1 0)
+			(at 25.4 38.1 0)
 			(hide yes)
 			(show_name no)
@@
 		)
 		(property "Description" "Power symbol creates a global label with name \"GND\" , ground"
-			(at 33.02 38.1 0)
+			(at 25.4 38.1 0)
 			(hide yes)
 			(show_name no)
@@
 			)
 		)
-		(property "Value" "100K"
+		(property "Value" "1k"
 			(at 40.64 52.0699 0)
 			(show_name no)
@@
 			)
 		)
-		(property "Footprint" "Resistor_SMD:R_0805_2012Metric_Pad1.20x1.40mm_HandSolder"
+		(property "Footprint" "Resistor_SMD:R_0603_1608Metric_Pad0.98x0.95mm_HandSolder"
 			(at 36.322 50.8 90)
 			(hide yes)
@@
 			)
 		)
-		(property "Footprint" "Resistor_SMD:R_0805_2012Metric_Pad1.20x1.40mm_HandSolder"
+		(property "Footprint" "Resistor_SMD:R_0603_1608Metric_Pad0.98x0.95mm_HandSolder"
 			(at 74.422 43.18 90)
 			(hide yes)
