File: Inda_Kidcad/Inda_Kidcad.kicad_sch (KiCad schematic)
At the start: 66 parts, among them J1 SERIALWIRE, J10 Conn_01x03_Pin, J15 Conn_01x02_Pin, J16 Conn_01x01_Pin, J17 Conn_01x01_Pin, J19 Conn_01x02_Pin, J2 LIPO, J20 Conn_01x02_Pin, J21 Conn_01x03_Pin, J22 Conn_01x03_Pin, J23 Conn_01x02_Pin, J24 Conn_01x02_Pin, J25 Conn_01x02_Pin, J3 BRIDGE, J8 Conn_01x02_Pin, J9 Conn_01x02_Pin, Q5 AO3401A, Q6 AO3401A, SW1 SW_Push, SW2 SW_Push, SW3 SW_Push_SPDT, SW4 SW_Push, SW5 SW_Push, SW6 SW_Push, U1 STM32f103C8t6, U12 vs1838, Y2 8Mhz

Commit message: Version 2 De Sumo Inda
Parts:
- removed D5: 12V, Resistor_SMD:R_1206_3216Metric_Pad1.30x1.75mm_HandSolder, symbol Device:D_Zener
- removed D6: GREEN, LED_SMD:LED_1206_3216Metric_Pad1.42x1.75mm_HandSolder, symbol Device:LED
- removed J16, J17: Conn_01x01_Pin, Footprint:pad_1_SMD, symbol Connector:Conn_01x01_Pin
- removed J19, J20: Conn_01x02_Pin, Footprint:Molex Header 2 hole 2.54mm, symbol Connector:Conn_01x02_Pin
- removed J2: LIPO, Connector_Molex:Molex_SL_171971-0002_1x02_P2.54mm_Vertical, symbol Connector:Conn_01x02_Pin
- removed J24: Conn_01x02_Pin, Footprint:CONN_SMD_01X02_IR, symbol Connector:Conn_01x02_Pin
- removed J3: BRIDGE, Connector_PinHeader_2.54mm:PinHeader_1x02_P2.54mm_Vertical, symbol Connector:Conn_01x02_Pin
- removed Q5, Q6: AO3401A, Package_TO_SOT_SMD:SOT-23, symbol Transistor_FET:AO3401A
- removed R18, R19: 100K, Resistor_SMD:R_0805_2012Metric_Pad1.20x1.40mm_HandSolder, symbol Device:R
- removed R20: 20K, Resistor_SMD:R_0805_2012Metric_Pad1.20x1.40mm_HandSolder, symbol Device:R
- removed SW3: SW_Push_SPDT, Button_Switch_SMD:SW_SPDT_PCM12, symbol Switch:SW_Push_SPDT
- U1: symbol Micromouse_Library:STM32F103C8T6 -> LIB_MCU:STM32F103C8T6
- U12: symbol Micromouse_Library:1838 -> LIB_Componentes:1838_ALIEXPRESS
Connections:
- net CURRENT_MOTL: no longer names the net of U1.15 (PA5_ADC5_SCK1)
- net CURRENT_MOTR: no longer names the net of U1.16 (PA6_ADC6_MISO1_PWM3)
- net Mod_RX4: no longer names the net of U1.13 (PA3_ADC3_RX2_PWM2)
- net Mod_TX4: no longer names the net of R3.1, U1.20 (PB2)
- no-connect marks 6 -> 8
Other:
- sheet Motores renamed MOTOR
- sheet sensores_linea renamed SENSOR_LINEA
- removed sheet INFRAROJOS
- sheet ALIMENTACION ports: added none; removed VIN
- sheet MOTOR ports: added none; removed CURRENT_MOTL, CURRENT_MOTR, MOTA_L, MOTA_R, MOTB_L, MOTB_R
- moved on the sheet: H1, H2, H3, H4, J25, R3, R42, R43

Commit message: Se cambia simbolos como huellas, se coloca solo mosfet para interruptor y se empieza con pcb
Parts:
- removed J1: SERIALWIRE, Connector_IDC:IDC-Header_2x03_P2.54mm_Vertical, symbol Connector_Generic:Conn_02x03_Odd_Even
- removed J10: Conn_01x03_Pin, Footprint:CONN_SMD_01X03_IR, symbol Connector:Conn_01x03_Pin
- removed J15, J23, J25, J8, J9: Conn_01x02_Pin, Footprint:CONN_SMD_01X02_IR, symbol Connector:Conn_01x02_Pin
- removed J21, J22: Conn_01x03_Pin, Connector_PinHeader_2.54mm:PinHeader_1x03_P2.54mm_Vertical, symbol Connector:Conn_01x03_Pin
- added J1: SWD_UART_CONN, Connector_IDC:IDC-Header_2x03_P2.54mm_Vertical, symbol LIB_CONECTORES:SWD_UART_CONN_6P
- added J2: Conn_01x03, symbol Connector_Generic:Conn_01x03
- added J3: Conn_01x03, Connector_PinHeader_2.54mm:PinHeader_1x03_P2.54mm_Vertical, symbol Connector_Generic:Conn_01x03
- added J4: Conn_01x02, symbol Connector_Generic:Conn_01x02
- added J6: Conn_01x04, symbol Connector_Generic:Conn_01x04
- U2: renamed from U12; footprint Connector_PinHeader_2.54mm:PinHeader_1x03_P2.54mm_Vertical -> Footprint:1838_aliexpress
- renumbered C8 to C1, C37 to C10, C38 to C11, C5 to C2, C7 to C3, C9 to C4, C3 to C5, C1 to C6, C2 to C7, C4 to C8, C6 to C9, D7 to D1, D8 to D2, D9 to D3, D10 to D4, R35 to R10, R37 to R11, R38 to R12, R3 to R13, R40 to R14, R41 to R15, R42 to R3, R43 to R4, R32 to R5, R33 to R6, R36 to R7, R39 to R8, R34 to R9, SW4 to SW3, SW5 to SW4, SW6 to SW5, Y2 to Y1
Connections:
- net +3.3V: now also J1.1 (VAPP), J4.2 (Pin_2)
- net +5V: now also J3.2 (Pin_2)
- net GND: now also J1.2 (GND), J3.1 (Pin_1), J4.1 (Pin_1)
- net Linea1: now also J2.1 (Pin_1)
- net Linea2: now also J2.2 (Pin_2)
- net Linea3: now also J2.3 (Pin_3)
- net RX: now also J1.3 (RX)
- net SERVO: now also J3.3 (Pin_3)
- net SWCLK: now also J1.6 (SWCLK)
- net SWDIO: now also J1.4 (SWDIO)
- net TX: now also J1.5 (TX)
- net SHARP_A4: now reaches U1.13 (PA3_ADC3_RX2_PWM2)
- net SHARP_A4: now also J6.4 (Pin_4)
- net EN_MOT: no longer names the net of U1.33 (PA12_USB++)
- net Mod_RX1 renamed SHARP_A1
- net SHARP_A1: now also J6.1 (Pin_1)
- net Mod_RX2 renamed SHARP_A2
- net SHARP_A2: now also J6.2 (Pin_2)
- net Mod_RX3 renamed SHARP_A3
- net SHARP_A3: now also J6.3 (Pin_3)
- net Mod_TX1: no longer names the net of U1.25 (PB12_SS2)
- no-connect marks 8 -> 9
Other:
- sheet ALIMENTACION ports: added VBAT; removed none
- sheet MOTOR ports: added none; removed EN_MOT
- moved on the sheet: C10, C11, C2, C3, C4, C5, C6, C7, C8, C9, D1, D2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

Commit message: Se corrigio pcb y se agrego conectores molex a sensores
Parts:
- J2: footprint (none) -> Connector_Molex:Molex_KK-254_AE-6410-03A_1x03_P2.54mm_Vertical
- J4: footprint (none) -> Connector_Molex:Molex_KK-254_AE-6410-02A_1x02_P2.54mm_Vertical
- J6: footprint (none) -> Connector_Molex:Molex_KK-254_AE-6410-04A_1x04_P2.54mm_Vertical
Changed lines of the file:
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@@
 			)
 		)
-		(property "Footprint" ""
+		(property "Footprint" "Connector_Molex:Molex_KK-254_AE-6410-02A_1x02_P2.54mm_Vertical"
 			(at 261.62 144.78 0)
 			(hide yes)
@@
 			)
 		)
-		(property "Footprint" ""
+		(property "Footprint" "Connector_Molex:Molex_KK-254_AE-6410-03A_1x03_P2.54mm_Vertical"
 			(at 261.62 157.48 0)
 			(hide yes)
@@
 			)
 		)
-		(property "Footprint" ""
+		(property "Footprint" "Connector_Molex:Molex_KK-254_AE-6410-04A_1x04_P2.54mm_Vertical"
 			(at 177.8 160.02 0)
 			(hide yes)

Commit message: Se ruteo y se cambio conectores a jst ph 2mm
Parts:
- J2: footprint Connector_Molex:Molex_KK-254_AE-6410-03A_1x03_P2.54mm_Vertical -> Connector_JST:JST_PH_S3B-PH-K_1x03_P2.00mm_Horizontal
- J3: footprint Connector_PinHeader_2.54mm:PinHeader_1x03_P2.54mm_Vertical -> Connector_PinHeader_2.54mm:PinHeader_1x03_P2.54mm_Horizontal
- J4: footprint Connector_Molex:Molex_KK-254_AE-6410-02A_1x02_P2.54mm_Vertical -> Connector_JST:JST_PH_S2B-PH-K_1x02_P2.00mm_Horizontal
- J6: footprint Connector_Molex:Molex_KK-254_AE-6410-04A_1x04_P2.54mm_Vertical -> Connector_JST:JST_PH_S4B-PH-K_1x04_P2.00mm_Horizontal
Connections:
- net +3.3V: now also D1.2 (A), D2.2 (A), D3.2 (A), D4.2 (A); no longer J4.2 (Pin_2)
- net GND: now also J4.2 (Pin_2); no longer D1.1 (K), D2.1 (K), D3.1 (K), D4.1 (K), J4.1 (Pin_1)
- net LED1: now also U1.4 (PC15_OSC32K_B); no longer U1.46 (PB9_PWM4)
- net LED2: now also U1.3 (PC14_OSC32K_A); no longer U1.2 (PC13)
- net LED3: now also U1.2 (PC13); no longer U1.3 (PC14_OSC32K_A)
- net LED4: now also U1.46 (PB9_PWM4); no longer U1.4 (PC15_OSC32K_B)
- net PWMA_MOTL: now also U1.29 (PA8_PWM1); no longer U1.32 (PA11_USB--_PWM1)
- net PWMA_MOTR: now also U1.31 (PA10_RX1_PWM1); no longer U1.30 (PA9_TX1_PWM1)
- net PWMB_MOTL: now also U1.30 (PA9_TX1_PWM1); no longer U1.31 (PA10_RX1_PWM1)
- net PWMB_MOTR: now also U1.32 (PA11_USB--_PWM1); no longer U1.29 (PA8_PWM1)
- net at R5.2: now also D1.1 (K); no longer D1.2 (A)
- net at R10.2: now also D4.1 (K); no longer D4.2 (A)
- net at R9.2: now also D3.1 (K); no longer D3.2 (A)
- net at R6.2: now also D2.1 (K); no longer D2.2 (A)
- new net +3V3: J4.1 (Pin_1)
Other:
- moved on the sheet: D1, D2, D3, D4

Commit message: rev 2.0 con 4 capas y terminada a falta de revision
Parts:
- SW3, SW4, SW5: footprint Button_Switch_SMD:SW_SPST_CK_RS282G05A3 -> Button_Switch_SMD:SW_Push_SPST_NO_Alps_SKRK
Changed lines of the file:
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@@
 			)
 		)
-		(property "Footprint" "Button_Switch_SMD:SW_SPST_CK_RS282G05A3"
+		(property "Footprint" "Button_Switch_SMD:SW_Push_SPST_NO_Alps_SKRK"
 			(at 135.89 158.75 0)
 			(hide yes)
@@
 			)
 		)
-		(property "Footprint" "Button_Switch_SMD:SW_SPST_CK_RS282G05A3"
+		(property "Footprint" "Button_Switch_SMD:SW_Push_SPST_NO_Alps_SKRK"
 			(at 151.13 158.75 0)
 			(hide yes)
@@
 			)
 		)
-		(property "Footprint" "Button_Switch_SMD:SW_SPST_CK_RS282G05A3"
+		(property "Footprint" "Button_Switch_SMD:SW_Push_SPST_NO_Alps_SKRK"
 			(at 120.65 158.75 0)
 			(hide yes)

Commit message: Terminado mini sumo v2 a espera de revision
Connections:
- net Mod_TX2: no longer names the net of U1.18 (PB0_ADC8_PWM3)
- net Mod_TX3: no longer names the net of U1.19 (PB1_ADC9_PWM3)
- no-connect marks 9 -> 11
Changed lines of the file:
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@@
+	)
+	(no_connect
+		(at 213.36 97.79)
 	)
 	(no_connect
@@
 		(at 260.35 83.82)
 	)
+	(no_connect
+		(at 209.55 97.79)
+	)
 	(wire
 		(pts
@@
 		(pts
 			(xy 40.64 33.02) (xy 40.64 35.56)
-		)
-		(stroke
-			(width 0)
-			(type default)
-		)
-	)
-	(wire
-		(pts
-			(xy 209.55 97.79) (xy 209.55 107.95)
-		)
-		(stroke
-			(width 0)
-			(type default)
-		)
-	)
-	(wire
-		(pts
-			(xy 213.36 97.79) (xy 213.36 107.95)
 		)
 		(stroke
@@
 		)
 	)
-	(label "Mod_TX3"
-		(at 213.36 107.95 90)
-		(effects
-			(font
-				(size 1.27 1.27)
-			)
-			(justify left bottom)
-		)
-	)
 	(label "OSC_B"
 		(at 20.32 21.59 180)
@@
 		(effects
 			(font
-				(size 1.27 1.27)
-			)
-			(justify left bottom)
-		)
-	)
-	(label "Mod_TX2"
-		(at 209.55 107.95 90)
-		(effects
-			(font

Commit message: cambios ultimos
Parts:
- R1, R13, R2: footprint Capacitor_SMD:C_0805_2012Metric_Pad1.18x1.45mm_HandSolder -> Resistor_SMD:R_0603_1608Metric_Pad0.98x0.95mm_HandSolder
- R10, R11, R12, R14, R15, R3, R4, R5, R6, R7, R8, R9: footprint Resistor_SMD:R_0805_2012Metric_Pad1.20x1.40mm_HandSolder -> Resistor_SMD:R_0603_1608Metric_Pad0.98x0.95mm_HandSolder
Changed lines of the file:
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@@
 			)
 		)
-		(property "Footprint" "Resistor_SMD:R_0805_2012Metric_Pad1.20x1.40mm_HandSolder"
+		(property "Footprint" "Resistor_SMD:R_0603_1608Metric_Pad0.98x0.95mm_HandSolder"
 			(at 112.522 118.11 90)
 			(hide yes)
@@
 			)
 		)
-		(property "Footprint" "Capacitor_SMD:C_0805_2012Metric_Pad1.18x1.45mm_HandSolder"
+		(property "Footprint" "Resistor_SMD:R_0603_1608Metric_Pad0.98x0.95mm_HandSolder"
 			(at 29.972 67.31 90)
 			(hide yes)
@@
 			)
 		)
-		(property "Footprint" "Resistor_SMD:R_0805_2012Metric_Pad1.20x1.40mm_HandSolder"
+		(property "Footprint" "Resistor_SMD:R_0603_1608Metric_Pad0.98x0.95mm_HandSolder"
 			(at 140.462 118.11 90)
 			(hide yes)
@@
 			)
 		)
-		(property "Footprint" "Resistor_SMD:R_0805_2012Metric_Pad1.20x1.40mm_HandSolder"
+		(property "Footprint" "Resistor_SMD:R_0603_1608Metric_Pad0.98x0.95mm_HandSolder"
 			(at 79.502 110.49 90)
 			(hide yes)
@@
 			)
 		)
-		(property "Footprint" "Resistor_SMD:R_0805_2012Metric_Pad1.20x1.40mm_HandSolder"
+		(property "Footprint" "Resistor_SMD:R_0603_1608Metric_Pad0.98x0.95mm_HandSolder"
 			(at 123.952 181.61 90)
 			(hide yes)
@@
 			)
 		)
-		(property "Footprint" "Resistor_SMD:R_0805_2012Metric_Pad1.20x1.40mm_HandSolder"
+		(property "Footprint" "Resistor_SMD:R_0603_1608Metric_Pad0.98x0.95mm_HandSolder"
 			(at 120.142 60.96 90)
 			(hide yes)
@@
 			)
 		)
-		(property "Footprint" "Capacitor_SMD:C_0805_2012Metric_Pad1.18x1.45mm_HandSolder"
+		(property "Footprint" "Resistor_SMD:R_0603_1608Metric_Pad0.98x0.95mm_HandSolder"
 			(at 215.392 109.22 90)
 			(hide yes)
@@
 			)
 		)
-		(property "Footprint" "Resistor_SMD:R_0805_2012Metric_Pad1.20x1.40mm_HandSolder"
+		(property "Footprint" "Resistor_SMD:R_0603_1608Metric_Pad0.98x0.95mm_HandSolder"
 			(at 127.762 60.96 90)
 			(hide yes)
@@
 			)
 		)
-		(property "Footprint" "Capacitor_SMD:C_0805_2012Metric_Pad1.18x1.45mm_HandSolder"
+		(property "Footprint" "Resistor_SMD:R_0603_1608Metric_Pad0.98x0.95mm_HandSolder"
 			(at 59.182 83.82 90)
 			(hide yes)
@@
 			)
 		)
-		(property "Footprint" "Resistor_SMD:R_0805_2012Metric_Pad1.20x1.40mm_HandSolder"
+		(property "Footprint" "Resistor_SMD:R_0603_1608Metric_Pad0.98x0.95mm_HandSolder"
 			(at 79.502 99.06 90)
 			(hide yes)
@@
 			)
 		)
-		(property "Footprint" "Resistor_SMD:R_0805_2012Metric_Pad1.20x1.40mm_HandSolder"
+		(property "Footprint" "Resistor_SMD:R_0603_1608Metric_Pad0.98x0.95mm_HandSolder"
 			(at 139.192 170.18 90)
 			(hide yes)
@@
 			)
 		)
-		(property "Footprint" "Resistor_SMD:R_0805_2012Metric_Pad1.20x1.40mm_HandSolder"
+		(property "Footprint" "Resistor_SMD:R_0603_1608Metric_Pad0.98x0.95mm_HandSolder"
 			(at 154.432 170.18 90)
 			(hide yes)
@@
 			)
 		)
-		(property "Footprint" "Resistor_SMD:R_0805_2012Metric_Pad1.20x1.40mm_HandSolder"
+		(property "Footprint" "Resistor_SMD:R_0603_1608Metric_Pad0.98x0.95mm_HandSolder"
 			(at 123.952 170.18 90)
 			(hide yes)
@@
 			)
 		)
-		(property "Footprint" "Resistor_SMD:R_0805_2012Metric_Pad1.20x1.40mm_HandSolder"
+		(property "Footprint" "Resistor_SMD:R_0603_1608Metric_Pad0.98x0.95mm_HandSolder"
 			(at 130.302 118.11 90)
 			(hide yes)
@@
 			)
 		)
-		(property "Footprint" "Resistor_SMD:R_0805_2012Metric_Pad1.20x1.40mm_HandSolder"
+		(property "Footprint" "Resistor_SMD:R_0603_1608Metric_Pad0.98x0.95mm_HandSolder"
 			(at 121.412 118.11 90)
 			(hide yes)
