File: Inda_Kidcad/sensores_linea.kicad_sch (KiCad schematic)
At the start: 20 parts, among them J4 Conn_01x03_Pin, J5 Conn_01x03_Pin, J6 Conn_01x03_Pin, J7 Conn_01x03_Pin, U10 QRE111GR, U11 QRE111GR, U8 QRE111GR, U9 QRE111GR

Commit message: Version 2 De Sumo Inda
Parts:
- removed C36: 100nF, Capacitor_SMD:C_0603_1608Metric_Pad1.08x0.95mm_HandSolder, symbol Device:C
- removed J7: Conn_01x03_Pin, Footprint:CONN_SMD_01X03_IR, symbol Connector:Conn_01x03_Pin
- removed R30: 150, Resistor_SMD:R_0805_2012Metric_Pad1.20x1.40mm_HandSolder, symbol Device:R
- removed R31: 15k, Resistor_SMD:R_0805_2012Metric_Pad1.20x1.40mm_HandSolder, symbol Device:R
- removed U11: QRE111GR, Footprint:QRE1113GR_IR, symbol Micromouse_Library:QRE1113GR
- U10, U8, U9: symbol Micromouse_Library:QRE1113GR -> LIB_Componentes:QRE1113GR
Other:
- moved on the sheet: C33, C34, C35, J4, J5, J6, R26, R27, R28, R29

Commit message: Se cambia simbolos como huellas, se coloca solo mosfet para interruptor y se empieza con pcb
Parts:
- renumbered C33 to C26, C34 to C27, C35 to C28, J5 to J13, J4 to J14, J6 to J15, R24 to R22, R25 to R23, R26 to R24, R27 to R25, R28 to R26, R29 to R27
Changed lines of the file:
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@@
 		(dnp no)
 		(fields_autoplaced yes)
-		(property "Reference" "C33"
+		(property "Reference" "C26"
 			(at 45.72 74.9299 0)
 			(show_name no)
@@
 			(project "Inda_Kidcad"
 				(path "/0fd92b06-954d-41bf-a53b-1bc8635b69f8/5718c1eb-8efd-49e8-a054-b8ab45346b8a"
-					(reference "C33")
+					(reference "C26")
 					(unit 1)
 				)
@@
 		(dnp no)
 		(fields_autoplaced yes)
-		(property "Reference" "J6"
+		(property "Reference" "J15"
 			(at 155.575 52.07 0)
 			(show_name no)
@@
 			(project "Inda_Kidcad"
 				(path "/0fd92b06-954d-41bf-a53b-1bc8635b69f8/5718c1eb-8efd-49e8-a054-b8ab45346b8a"
-					(reference "J6")
+					(reference "J15")
 					(unit 1)
 				)
@@
 		(dnp no)
 		(fields_autoplaced yes)
-		(property "Reference" "J5"
+		(property "Reference" "J13"
 			(at 37.465 49.53 0)
 			(show_name no)
@@
 			(project "Inda_Kidcad"
 				(path "/0fd92b06-954d-41bf-a53b-1bc8635b69f8/5718c1eb-8efd-49e8-a054-b8ab45346b8a"
-					(reference "J5")
+					(reference "J13")
 					(unit 1)
 				)
@@
 		(dnp no)
 		(fields_autoplaced yes)
-		(property "Reference" "R29"
+		(property "Reference" "R27"
 			(at 176.53 29.2099 0)
 			(show_name no)
@@
 			(project "Inda_Kidcad"
 				(path "/0fd92b06-954d-41bf-a53b-1bc8635b69f8/5718c1eb-8efd-49e8-a054-b8ab45346b8a"
-					(reference "R29")
+					(reference "R27")
 					(unit 1)
 				)
@@
 		(dnp no)
 		(fields_autoplaced yes)
-		(property "Reference" "R28"
+		(property "Reference" "R26"
 			(at 152.4 29.2099 0)
 			(show_name no)
@@
 			(project "Inda_Kidcad"
 				(path "/0fd92b06-954d-41bf-a53b-1bc8635b69f8/5718c1eb-8efd-49e8-a054-b8ab45346b8a"
-					(reference "R28")
+					(reference "R26")
 					(unit 1)
 				)
@@
 		(dnp no)
 		(fields_autoplaced yes)
-		(property "Reference" "R27"
+		(property "Reference" "R25"
 			(at 116.84 27.9399 0)
 			(show_name no)
@@
 			(project "Inda_Kidcad"
 				(path "/0fd92b06-954d-41bf-a53b-1bc8635b69f8/5718c1eb-8efd-49e8-a054-b8ab45346b8a"
-					(reference "R27")
+					(reference "R25")
 					(unit 1)
 				)
@@
 		(dnp no)
 		(fields_autoplaced yes)
-		(property "Reference" "R25"
+		(property "Reference" "R23"
 			(at 57.15 29.2099 0)
 			(show_name no)
@@
 			(project "Inda_Kidcad"
 				(path "/0fd92b06-954d-41bf-a53b-1bc8635b69f8/5718c1eb-8efd-49e8-a054-b8ab45346b8a"
-					(reference "R25")
+					(reference "R23")
 					(unit 1)
 				)
@@
 		(dnp no)
 		(fields_autoplaced yes)
-		(property "Reference" "C35"
+		(property "Reference" "C28"
 			(at 165.1 73.6599 0)
 			(show_name no)
@@
 			(project "Inda_Kidcad"
 				(path "/0fd92b06-954d-41bf-a53b-1bc8635b69f8/5718c1eb-8efd-49e8-a054-b8ab45346b8a"
-					(reference "C35")
+					(reference "C28")
 					(unit 1)
 				)
@@
 		(dnp no)
 		(fields_autoplaced yes)
-		(property "Reference" "J4"
+		(property "Reference" "J14"
 			(at 95.885 50.8 0)
 			(show_name no)
@@
 			(project "Inda_Kidcad"
 				(path "/0fd92b06-954d-41bf-a53b-1bc8635b69f8/5718c1eb-8efd-49e8-a054-b8ab45346b8a"
-					(reference "J4")
+					(reference "J14")
 					(unit 1)
 				)
@@
 		(dnp no)
 		(fields_autoplaced yes)
-		(property "Reference" "C34"
+		(property "Reference" "C27"
 			(at 97.79 76.1999 0)
 			(show_name no)
@@
 			(project "Inda_Kidcad"
 				(path "/0fd92b06-954d-41bf-a53b-1bc8635b69f8/5718c1eb-8efd-49e8-a054-b8ab45346b8a"
-					(reference "C34")
+					(reference "C27")
 					(unit 1)
 				)
@@
 		(dnp no)
 		(fields_autoplaced yes)
-		(property "Reference" "R24"
+		(property "Reference" "R22"
 			(at 33.02 29.2099 0)
 			(show_name no)
@@
 			(project "Inda_Kidcad"
 				(path "/0fd92b06-954d-41bf-a53b-1bc8635b69f8/5718c1eb-8efd-49e8-a054-b8ab45346b8a"
-					(reference "R24")
+					(reference "R22")
 					(unit 1)
 				)
@@
 		(dnp no)
 		(fields_autoplaced yes)
-		(property "Reference" "R26"
+		(property "Reference" "R24"
 			(at 92.71 27.9399 0)
 			(show_name no)
@@
 			(project "Inda_Kidcad"
 				(path "/0fd92b06-954d-41bf-a53b-1bc8635b69f8/5718c1eb-8efd-49e8-a054-b8ab45346b8a"
-					(reference "R26")
-					(unit 1)
-				)
+					(reference "R24")
+					(unit 1)
+				)

Commit message: rev 2.0 con 4 capas y terminada a falta de revision
Parts:
- R22, R23, R24, R25, R26, R27: footprint Resistor_SMD:R_0805_2012Metric_Pad1.20x1.40mm_HandSolder -> Resistor_SMD:R_0603_1608Metric
Changed lines of the file:
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@@
 			)
 		)
-		(property "Footprint" "Resistor_SMD:R_0805_2012Metric_Pad1.20x1.40mm_HandSolder"
+		(property "Footprint" "Resistor_SMD:R_0603_1608Metric"
 			(at 172.212 30.48 90)
 			(hide yes)
@@
 			)
 		)
-		(property "Footprint" "Resistor_SMD:R_0805_2012Metric_Pad1.20x1.40mm_HandSolder"
+		(property "Footprint" "Resistor_SMD:R_0603_1608Metric"
 			(at 148.082 30.48 90)
 			(hide yes)
@@
 			)
 		)
-		(property "Footprint" "Resistor_SMD:R_0805_2012Metric_Pad1.20x1.40mm_HandSolder"
+		(property "Footprint" "Resistor_SMD:R_0603_1608Metric"
 			(at 112.522 29.21 90)
 			(hide yes)
@@
 			)
 		)
-		(property "Footprint" "Resistor_SMD:R_0805_2012Metric_Pad1.20x1.40mm_HandSolder"
+		(property "Footprint" "Resistor_SMD:R_0603_1608Metric"
 			(at 52.832 30.48 90)
 			(hide yes)
@@
 			)
 		)
-		(property "Footprint" "Resistor_SMD:R_0805_2012Metric_Pad1.20x1.40mm_HandSolder"
+		(property "Footprint" "Resistor_SMD:R_0603_1608Metric"
 			(at 28.702 30.48 90)
 			(hide yes)
@@
 			)
 		)
-		(property "Footprint" "Resistor_SMD:R_0805_2012Metric_Pad1.20x1.40mm_HandSolder"
+		(property "Footprint" "Resistor_SMD:R_0603_1608Metric"
 			(at 88.392 29.21 90)
 			(hide yes)

Commit message: cambios ultimos
Parts:
- R22, R23, R24, R25, R26, R27: footprint Resistor_SMD:R_0603_1608Metric -> Resistor_SMD:R_0603_1608Metric_Pad0.98x0.95mm_HandSolder
Changed lines of the file:
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@@
 			)
 		)
-		(property "Footprint" "Resistor_SMD:R_0603_1608Metric"
+		(property "Footprint" "Resistor_SMD:R_0603_1608Metric_Pad0.98x0.95mm_HandSolder"
 			(at 172.212 30.48 90)
 			(hide yes)
@@
 			)
 		)
-		(property "Footprint" "Resistor_SMD:R_0603_1608Metric"
+		(property "Footprint" "Resistor_SMD:R_0603_1608Metric_Pad0.98x0.95mm_HandSolder"
 			(at 148.082 30.48 90)
 			(hide yes)
@@
 			)
 		)
-		(property "Footprint" "Resistor_SMD:R_0603_1608Metric"
+		(property "Footprint" "Resistor_SMD:R_0603_1608Metric_Pad0.98x0.95mm_HandSolder"
 			(at 112.522 29.21 90)
 			(hide yes)
@@
 			)
 		)
-		(property "Footprint" "Resistor_SMD:R_0603_1608Metric"
+		(property "Footprint" "Resistor_SMD:R_0603_1608Metric_Pad0.98x0.95mm_HandSolder"
 			(at 52.832 30.48 90)
 			(hide yes)
@@
 			)
 		)
-		(property "Footprint" "Resistor_SMD:R_0603_1608Metric"
+		(property "Footprint" "Resistor_SMD:R_0603_1608Metric_Pad0.98x0.95mm_HandSolder"
 			(at 28.702 30.48 90)
 			(hide yes)
@@
 			)
 		)
-		(property "Footprint" "Resistor_SMD:R_0603_1608Metric"
+		(property "Footprint" "Resistor_SMD:R_0603_1608Metric_Pad0.98x0.95mm_HandSolder"
 			(at 88.392 29.21 90)
 			(hide yes)
